Commit message: added a config file to localization_pkg, added configuration for Extended Kalman Filter, added an imu to gazebo test bot, and applied robot_localization pkg to gazebo test bot.

File: src/test_bot_description/urdf/test_bot.xacro (robot description, xacro)
@@ -85,8 +85,23 @@
 		<xacro:cylinder_inertia m="0.1" r="${lidar_radius}" h="${lidar_height}" xyz="0 0 0" rpy="0 0 0" />
 	</link>
+	<link name="imu_link">
+		<visual>
+			<geometry>
+			  <box size="0.05 0.05 0.05"/>
+			</geometry>
+			<origin xyz="0 0 0" rpy="0 0 0" />
+			<material name="green" />
+		</visual>
+		<collision>
+			<geometry>
+				<box size="0.05 0.05 0.05"/>
+			</geometry>
+		</collision>
+		<xacro:box_inertia m="0.1" l="0.05" w="0.05" h="0.05" xyz="0 0 0" rpy="0 0 0" />
+	</link>
 	<joint name="base_joint" type="fixed">
-		<parent link="base_footprint" />
-		<child link="base_link" />
-		<origin xyz="0 0 ${wheel_radius}" rpy="0 0 0" />
+		<parent link="base_link" />
+		<child link="base_footprint" />
+		<origin xyz="0 0 ${-wheel_radius}" rpy="0 0 0" />
 	</joint>
 	<joint name="base_rear_right_wheel_joint" type="continuous">
@@ -122,3 +137,8 @@
         <origin xyz="${(base_length/2) - lidar_radius} 0 ${base_height + (lidar_height/2)}" rpy="0 0 0" />
     </joint>
+	<joint name="base_imu_joint" type="fixed">
+		<parent link="base_link" />
+		<child link="imu_link" />
+		<origin xyz="0 0 ${base_height + 0.025}" rpy="0 0 0" />
+	</joint>
 </robot>

File: src/test_bot_description/urdf/test_bot_gazebo.xacro (robot description, xacro)
@@ -1,5 +1,4 @@
 <?xml version="1.0"?>
-<robot
-	xmlns:xacro="http://www.ros.org/wiki/xacro">
+<robot xmlns:xacro="http://www.ros.org/wiki/xacro">
 	<gazebo reference="Ebox_link">
 		<material>Gazebo/Grey</material>
@@ -50,6 +49,6 @@
             <plugin name="lidar_sensor_plugin" filename="libgazebo_ros_ray_sensor.so">
                 <ros>
-                  <!-- Configure namespace and remap to publish to /ray/pointcloud2 -->
-                  <namespace>/ray</namespace>
+                  <!-- Configure namespace and remap to publish to /lidar/pointcloud2 -->
+                  <namespace>/lidar</namespace>
                   <remapping>~/out:=pointcloud2</remapping>
                 </ros>
@@ -63,7 +62,76 @@
         </sensor>
     </gazebo>
+    <gazebo reference="imu_link">
+        <material>Gazebo/Green</material>
+        <sensor name="imu_sensor" type="imu">
+         <plugin filename="libgazebo_ros_imu_sensor.so" name="imu_plugin">
+            <ros>
+              <namespace>/imu_link</namespace>
+              <remapping>~/out:=imu</remapping>
+            </ros>
+            <initial_orientation_as_reference>false</initial_orientation_as_reference>
+          </plugin>
+          <always_on>true</always_on>
+          <update_rate>100</update_rate>
+          <visualize>true</visualize>
+          <imu>
+            <angular_velocity>
+              <x>
+                <noise type="gaussian">
+                  <mean>0.0</mean>
+                  <stddev>2e-4</stddev>
+                  <bias_mean>0.0000075</bias_mean>
+                  <bias_stddev>0.0000008</bias_stddev>
+                </noise>
+              </x>
+              <y>
+                <noise type="gaussian">
+                  <mean>0.0</mean>
+                  <stddev>2e-4</stddev>
+                  <bias_mean>0.0000075</bias_mean>
+                  <bias_stddev>0.0000008</bias_stddev>
+                </noise>
+              </y>
+              <z>
+                <noise type="gaussian">
+                  <mean>0.0</mean>
+                  <stddev>2e-4</stddev>
+                  <bias_mean>0.0000075</bias_mean>
+                  <bias_stddev>0.0000008</bias_stddev>
+                </noise>
+              </z>
+            </angular_velocity>
+            <linear_acceleration>
+              <x>
+                <noise type="gaussian">
+                  <mean>0.0</mean>
+                  <stddev>1.7e-2</stddev>
+                  <bias_mean>0.1</bias_mean>
+                  <bias_stddev>0.001</bias_stddev>
+                </noise>
+              </x>
+              <y>
+                <noise type="gaussian">
+                  <mean>0.0</mean>
+                  <stddev>1.7e-2</stddev>
+                  <bias_mean>0.1</bias_mean>
+                  <bias_stddev>0.001</bias_stddev>
+                </noise>
+              </y>
+              <z>
+                <noise type="gaussian">
+                  <mean>0.0</mean>
+                  <stddev>1.7e-2</stddev>
+                  <bias_mean>0.1</bias_mean>
+                  <bias_stddev>0.001</bias_stddev>
+                </noise>
+              </z>
+            </linear_acceleration>
+          </imu>
+        </sensor>
+    </gazebo>
 	<gazebo>
 		<plugin name="diff_drive_controller" filename="libgazebo_ros_diff_drive.so">
-			<!-- Update rate in Hz -->
+            <!-- Update rate in Hz -->
 			<update_rate>50</update_rate>
 			<!-- wheels -->
@@ -85,5 +153,5 @@
 			<odometry_topic>odom</odometry_topic>
 			<odometry_frame>odom</odometry_frame>
-			<robot_base_frame>base_footprint</robot_base_frame>
+			<robot_base_frame>base_link</robot_base_frame>
 		</plugin>
 	</gazebo>

Commit message: added depth camera and updated world

File: src/test_bot_description/urdf/test_bot.xacro (robot description, xacro)
@@ -4,15 +4,37 @@
 	<xacro:include filename="common_properties.xacro" />
 	<xacro:include filename="test_bot_gazebo.xacro" />
-	<xacro:property name="base_length" value="1.0" />
-	<xacro:property name="base_width" value="0.5" />
-	<xacro:property name="base_height" value="0.08" />
-	<xacro:property name="wheel_radius" value="0.15" />
-	<xacro:property name="wheel_length" value="0.1" />
+	<xacro:property name="base_length"
+		value="0.8" />
+	<xacro:property name="base_width"
+		value="0.4" />
+	<xacro:property name="base_height"
+		value="0.08" />
+	<xacro:property name="wheel_radius"
+		value="0.12" />
+	<xacro:property name="wheel_length"
+		value="0.08" />
 	<!--Ebox = Electrical box-->
-	<xacro:property name="Ebox_length" value="0.1" />
-	<xacro:property name="Ebox_width" value="0.5" />
-	<xacro:property name="Ebox_height" value="0.3" />
-    <xacro:property name="lidar_radius" value="0.04" />
-	<xacro:property name="lidar_height" value="0.04" />
+	<xacro:property name="Ebox_length"
+		value="0.1" />
+	<xacro:property name="Ebox_width"
+		value="0.4" />
+	<xacro:property name="Ebox_height"
+		value="0.25" />
+	<xacro:property name="lidar_radius"
+		value="0.04" />
+	<xacro:property name="lidar_height"
+		value="0.04" />
+	<xacro:property name="camera_length"
+		value="0.015" />
+	<xacro:property name="camera_width"
+		value="0.130" />
+	<xacro:property name="camera_height"
+		value="0.022" />
+	<xacro:property name="camera_pole_length"
+		value="0.02" />
+	<xacro:property name="camera_pole_width"
+		value="0.02" />
+	<xacro:property name="camera_pole_height"
+		value="0.2" />
 	<link name="base_footprint" />
 	<link name="base_link">
@@ -21,5 +43,6 @@
 				<box size="${base_length} ${base_width} ${base_height}" />
 			</geometry>
-			<origin xyz="0 0 ${base_height / 2}" rpy="0 0 0" />
+			<origin xyz="0 0 ${base_height / 2}"
+				rpy="0 0 0" />
 			<material name="grey" />
 		</visual>
@@ -28,24 +51,39 @@
 				<box size="${base_length} ${base_width} ${base_height}" />
 			</geometry>
-			<origin xyz="0 0 ${base_height / 2}" rpy="0 0 0" />
-		</collision>
-		<xacro:box_inertia m="7.0" l="${base_length}" w="${base_width}" h="${base_height}" xyz="0 0 ${base_height / 2}" rpy="0 0 0" />
-	</link>
-	<xacro:macro name="wheel_link" params="prefix">
+			<origin xyz="0 0 ${base_height / 2}"
+				rpy="0 0 0" />
+		</collision>
+		<xacro:box_inertia m="7.0"
+			l="${base_length}"
+			w="${base_width}"
+			h="${base_height}"
+			xyz="0 0 ${base_height / 2}"
+			rpy="0 0 0" />
+	</link>
+	<xacro:macro name="wheel_link"
+		params="prefix">
 		<link name="${prefix}_wheel_link">
 			<visual>
 				<geometry>
-					<cylinder radius="${wheel_radius}" length="${wheel_length}" />
+					<cylinder radius="${wheel_radius}"
+						length="${wheel_length}" />
 				</geometry>
-				<origin xyz="0 0 0" rpy="${pi / 2.0} 0 0" />
+				<origin xyz="0 0 0"
+					rpy="${pi / 2.0} 0 0" />
 				<material name="blue" />
 			</visual>
 			<collision>
 				<geometry>
-					<cylinder radius="${wheel_radius}" length="${wheel_length}" />
+					<cylinder radius="${wheel_radius}"
+						length="${wheel_length}" />
 				</geometry>
-				<origin xyz="0 0 0" rpy="${pi / 2.0} 0 0" />
+				<origin xyz="0 0 0"
+					rpy="${pi / 2.0} 0 0" />
 			</collision>
-			<xacro:cylinder_inertia m="1.5" r="${wheel_radius}" h="${wheel_length}" xyz="0 0 0" rpy="${pi / 2.0} 0 0" />
+			<xacro:cylinder_inertia m="1.5"
+				r="${wheel_radius}"
+				h="${wheel_length}"
+				xyz="0 0 0"
+				rpy="${pi / 2.0} 0 0" />
 		</link>
 	</xacro:macro>
@@ -59,5 +97,6 @@
 				<box size="${Ebox_length} ${Ebox_width} ${Ebox_height}" />
 			</geometry>
-			<origin xyz="0 0 0" rpy="0 0 0" />
+			<origin xyz="0 0 0"
+				rpy="0 0 0" />
 			<material name="grey" />
 		</visual>
@@ -66,79 +105,180 @@
 				<box size="${Ebox_length} ${Ebox_width} ${Ebox_height}" />
 			</geometry>
-			<origin xyz="0 0 0" rpy="0 0 0" />
-		</collision>
-		<xacro:box_inertia m="2.0" l="${Ebox_length}" w="${Ebox_width}" h="${Ebox_height}" xyz="0 0 0" rpy="0 0 0" />
+			<origin xyz="0 0 0"
+				rpy="0 0 0" />
+		</collision>
+		<xacro:box_inertia m="2.0"
+			l="${Ebox_length}"
+			w="${Ebox_width}"
+			h="${Ebox_height}"
+			xyz="0 0 0"
+			rpy="0 0 0" />
+	</link>
+	<link name="camera_pole_link">
+		<visual>
+			<geometry>
+				<box size="${camera_pole_length} ${camera_pole_width} ${camera_pole_height}" />
+			</geometry>
+			<origin xyz="0 0 0"
+				rpy="0 0 0" />
+			<material name="grey" />
+		</visual>
+		<collision>
+			<geometry>
+				<box size="${camera_pole_length} ${camera_pole_width} ${camera_pole_height}" />
+			</geometry>
+			<origin xyz="0 0 0"
+				rpy="0 0 0" />
+		</collision>
+		<xacro:box_inertia m="1.0"
+			l="${camera_pole_length}"
+			w="${camera_pole_width}"
+			h="${camera_pole_height}"
+			xyz="0 0 0"
+			rpy="0 0 0" />
 	</link>
 	<link name="lidar_link">
 		<visual>
 			<geometry>
-				<cylinder radius="${lidar_radius}" length="${lidar_height}" />
-			</geometry>
-            <origin xyz="0 0 0" rpy="0 0 0" />
+				<cylinder radius="${lidar_radius}"
+					length="${lidar_height}" />
+			</geometry>
+			<origin xyz="0 0 0"
+				rpy="0 0 0" />
 			<material name="green" />
 		</visual>
 		<collision>
 			<geometry>
-				<cylinder radius="${lidar_radius}" length="${lidar_height}" />
-			</geometry>
-		</collision>
-		<xacro:cylinder_inertia m="0.1" r="${lidar_radius}" h="${lidar_height}" xyz="0 0 0" rpy="0 0 0" />
-	</link>
+				<cylinder radius="${lidar_radius}"
+					length="${lidar_height}" />
+			</geometry>
+		</collision>
+		<xacro:cylinder_inertia m="0.1"
+			r="${lidar_radius}"
+			h="${lidar_height}"
+			xyz="0 0 0"
+			rpy="0 0 0" />
+	</link>
+	<link name="camera_link">
+		<visual>
+			<origin xyz="0 0 0"
+				rpy="0 0 0" />
+			<geometry>
+				<box size="${camera_length} ${camera_width} ${camera_height}" />
+			</geometry>
+			<material name="green" />
+		</visual>
+		<collision>
+			<origin xyz="0 0 0"
+				rpy="0 0 0" />
+			<geometry>
+				<box size="${camera_length} ${camera_width} ${camera_height}" />
+			</geometry>
+		</collision>
+		<xacro:box_inertia m="0.1"
+			l="${camera_length}"
+			w="${camera_width}"
+			h="${camera_height}"
+			xyz="0 0 0"
+			rpy="0 0 0" />
+	</link>
+	<link name="camera_depth_frame"/>
 	<link name="imu_link">
 		<visual>
 			<geometry>
-			  <box size="0.05 0.05 0.05"/>
-			</geometry>
-			<origin xyz="0 0 0" rpy="0 0 0" />
+				<box size="0.05 0.05 0.05" />
+			</geometry>
+			<origin xyz="0 0 0"
+				rpy="0 0 0" />
 			<material name="green" />
 		</visual>
 		<collision>
 			<geometry>
-				<box size="0.05 0.05 0.05"/>
-			</geometry>
-		</collision>
-		<xacro:box_inertia m="0.1" l="0.05" w="0.05" h="0.05" xyz="0 0 0" rpy="0 0 0" />
-	</link>
-	<joint name="base_joint" type="fixed">
+				<box size="0.05 0.05 0.05" />
+			</geometry>
+		</collision>
+		<xacro:box_inertia m="0.1"
+			l="0.05"
+			w="0.05"
+			h="0.05"
+			xyz="0 0 0"
+			rpy="0 0 0" />
+	</link>
+	<joint name="base_joint"
+		type="fixed">
 		<parent link="base_link" />
 		<child link="base_footprint" />
-		<origin xyz="0 0 ${-wheel_radius}" rpy="0 0 0" />
-	</joint>
-	<joint name="base_rear_right_wheel_joint" type="continuous">
+		<origin xyz="0 0 ${-wheel_radius}"
+			rpy="0 0 0" />
+	</joint>
+	<joint name="base_rear_right_wheel_joint"
+		type="continuous">
 		<parent link="base_link" />
 		<child link="rear_right_wheel_link" />
-		<origin xyz="${-base_length / 4.0} ${-(base_width + wheel_length) / 2.0} 0" rpy="0 0 0" />
+		<origin xyz="${-base_length / 4.0} ${-(base_width + wheel_length) / 2.0} 0"
+			rpy="0 0 0" />
 		<axis xyz="0 1 0" />
 	</joint>
-	<joint name="base_rear_left_wheel_joint" type="continuous">
+	<joint name="base_rear_left_wheel_joint"
+		type="continuous">
 		<parent link="base_link" />
 		<child link="rear_left_wheel_link" />
-		<origin xyz="${-base_length / 4.0} ${(base_width + wheel_length) / 2.0} 0" rpy="0 0 0" />
+		<origin xyz="${-base_length / 4.0} ${(base_width + wheel_length) / 2.0} 0"
+			rpy="0 0 0" />
 		<axis xyz="0 1 0" />
 	</joint>
-	<joint name="base_front_right_wheel_joint" type="fixed">
+	<joint name="base_front_right_wheel_joint"
+		type="fixed">
 		<parent link="base_link" />
 		<child link="front_right_wheel_link" />
-		<origin xyz="${base_length / 4.0} ${-(base_width + wheel_length) / 2.0} 0" rpy="0 0 0" />
-	</joint>
-	<joint name="base_front_left_wheel_joint" type="fixed">
+		<origin xyz="${base_length / 4.0} ${-(base_width + wheel_length) / 2.0} 0"
+			rpy="0 0 0" />
+	</joint>
+	<joint name="base_front_left_wheel_joint"
+		type="fixed">
 		<parent link="base_link" />
 		<child link="front_left_wheel_link" />
-		<origin xyz="${base_length / 4.0} ${(base_width + wheel_length) / 2.0} 0" rpy="0 0 0" />
-	</joint>
-	<joint name="base_Ebox_joint" type="fixed">
+		<origin xyz="${base_length / 4.0} ${(base_width + wheel_length) / 2.0} 0"
+			rpy="0 0 0" />
+	</joint>
+	<joint name="base_Ebox_joint"
+		type="fixed">
 		<parent link="base_link" />
 		<child link="Ebox_link" />
-		<origin xyz="${(-base_length / 2) - (Ebox_length / 2)} 0 ${Ebox_height / 2}" rpy="0 0 0" />
-	</joint>
-    <joint name="base_lidar_joint" type="fixed">
-        <parent link="base_link" />
-        <child link="lidar_link" />
-        <origin xyz="${(base_length/2) - lidar_radius} 0 ${base_height + (lidar_height/2)}" rpy="0 0 0" />
-    </joint>
-	<joint name="base_imu_joint" type="fixed">
+		<origin xyz="${(-base_length / 2) - (Ebox_length / 2)} 0 ${Ebox_height / 2}"
+			rpy="0 0 0" />
+	</joint>
+	<joint name="base_camera_pole_joint"
+		type="fixed">
+		<parent link="base_link" />
+		<child link="camera_pole_link" />
+		<origin xyz="${(base_length / 2) - (2*lidar_radius) - (camera_pole_length/2)} 0 ${(base_height/2) + (camera_pole_height/2)}"
+			rpy="0 0 0" />
+	</joint>
+	<joint name="base_lidar_joint"
+		type="fixed">
+		<parent link="base_link" />
+		<child link="lidar_link" />
+		<origin xyz="${(base_length/2) - lidar_radius} 0 ${base_height + (lidar_height/2)}"
+			rpy="0 0 0" />
+	</joint>
+	<joint name="base_camera_joint"
+		type="fixed">
+		<parent link="base_link" />
+		<child link="camera_link" />
+		<origin xyz="${(base_length / 2) - (2*lidar_radius) - (camera_pole_length/2)} 0 ${(base_height/2) + (camera_pole_height) + (camera_height/2)}"
+			rpy="0 0 0" />
+	</joint>
+	<joint name="camera_depth_joint" type="fixed">
+		<origin xyz="0 0 0" rpy="${-pi/2} 0 ${-pi/2}"/>
+		<parent link="camera_link"/>
+		<child link="camera_depth_frame"/>
+	  </joint>
+	<joint name="base_imu_joint"
+		type="fixed">
 		<parent link="base_link" />
 		<child link="imu_link" />
-		<origin xyz="0 0 ${base_height + 0.025}" rpy="0 0 0" />
+		<origin xyz="0 0 ${base_height + 0.025}"
+			rpy="0 0 0" />
 	</joint>
 </robot>
