Commit message: added depth camera and updated world

File: src/test_bot_description/urdf/test_bot_gazebo.xacro (robot description, xacro)
@@ -1,158 +1,200 @@
 <?xml version="1.0"?>
 <robot xmlns:xacro="http://www.ros.org/wiki/xacro">
-	<gazebo reference="Ebox_link">
-		<material>Gazebo/Grey</material>
-	</gazebo>
-	<gazebo reference="rear_right_wheel_link">
-		<material>Gazebo/Blue</material>
-	</gazebo>
-	<gazebo reference="rear_left_wheel_link">
-		<material>Gazebo/Blue</material>
-	</gazebo>
-	<gazebo reference="front_right_wheel_link">
-		<material>Gazebo/Blue</material>
-        <mu1 value="0.1"/>
-        <mu2 value="0.1"/>
-	</gazebo>
-	<gazebo reference="front_left_wheel_link">
-		<material>Gazebo/Blue</material>
-        <mu1 value="0.1" />
-        <mu2 value="0.1" />
-	</gazebo>
-    <gazebo reference="lidar_link">
-        <material>Gazebo/Green</material>
-        <sensor name="lidar_sensor" type="ray">
-            <pose>0 0 0 0 0 0</pose>
-            <visualize>true</visualize>
-            <update_rate>10.0</update_rate>
-            <ray>
-                <scan>
-                    <horizontal>
-                        <samples>720</samples>
-                        <resolution>1</resolution>
-                        <min_angle>-1.570796</min_angle>
-                        <max_angle>1.570796</max_angle>
-                    </horizontal>
-                </scan>
-                <range>
-                    <min>0.08</min>
-                    <max>10.0</max>
-                    <resolution>0.01</resolution>
-                </range>
-                <noise>
-                    <type>gaussian</type>
-                    <!-- Noise parameters based on your specific sensor -->
-                    <mean>0.0</mean>
-                    <stddev>0.01</stddev>
-                </noise>
-            </ray>
-            <plugin name="lidar_sensor_plugin" filename="libgazebo_ros_ray_sensor.so">
-                <ros>
-                  <!-- Configure namespace and remap to publish to /lidar/pointcloud2 -->
-                  <namespace>/lidar</namespace>
-                  <remapping>~/out:=pointcloud2</remapping>
-                </ros>
-                <!-- Output as a PointCloud2, see above for other types -->
-                <output_type>sensor_msgs/PointCloud2</output_type>
-                <!-- Clip intensity values so all are above 100, optional -->
-                <min_intensity>100.0</min_intensity>
-                <!-- Frame id for header of output, defaults to sensor's parent link name -->
-                <frame_name>lidar_link</frame_name>
-              </plugin>
-        </sensor>
-    </gazebo>
-    <gazebo reference="imu_link">
-        <material>Gazebo/Green</material>
-        <sensor name="imu_sensor" type="imu">
-         <plugin filename="libgazebo_ros_imu_sensor.so" name="imu_plugin">
-            <ros>
-              <namespace>/imu_link</namespace>
-              <remapping>~/out:=imu</remapping>
-            </ros>
-            <initial_orientation_as_reference>false</initial_orientation_as_reference>
-          </plugin>
-          <always_on>true</always_on>
-          <update_rate>100</update_rate>
-          <visualize>true</visualize>
-          <imu>
-            <angular_velocity>
-              <x>
-                <noise type="gaussian">
-                  <mean>0.0</mean>
-                  <stddev>2e-4</stddev>
-                  <bias_mean>0.0000075</bias_mean>
-                  <bias_stddev>0.0000008</bias_stddev>
-                </noise>
-              </x>
-              <y>
-                <noise type="gaussian">
-                  <mean>0.0</mean>
-                  <stddev>2e-4</stddev>
-                  <bias_mean>0.0000075</bias_mean>
-                  <bias_stddev>0.0000008</bias_stddev>
-                </noise>
-              </y>
-              <z>
-                <noise type="gaussian">
-                  <mean>0.0</mean>
-                  <stddev>2e-4</stddev>
-                  <bias_mean>0.0000075</bias_mean>
-                  <bias_stddev>0.0000008</bias_stddev>
-                </noise>
-              </z>
-            </angular_velocity>
-            <linear_acceleration>
-              <x>
-                <noise type="gaussian">
-                  <mean>0.0</mean>
-                  <stddev>1.7e-2</stddev>
-                  <bias_mean>0.1</bias_mean>
-                  <bias_stddev>0.001</bias_stddev>
-                </noise>
-              </x>
-              <y>
-                <noise type="gaussian">
-                  <mean>0.0</mean>
-                  <stddev>1.7e-2</stddev>
-                  <bias_mean>0.1</bias_mean>
-                  <bias_stddev>0.001</bias_stddev>
-                </noise>
-              </y>
-              <z>
-                <noise type="gaussian">
-                  <mean>0.0</mean>
-                  <stddev>1.7e-2</stddev>
-                  <bias_mean>0.1</bias_mean>
-                  <bias_stddev>0.001</bias_stddev>
-                </noise>
-              </z>
-            </linear_acceleration>
-          </imu>
-        </sensor>
-    </gazebo>
-	<gazebo>
-		<plugin name="diff_drive_controller" filename="libgazebo_ros_diff_drive.so">
-            <!-- Update rate in Hz -->
-			<update_rate>50</update_rate>
-			<!-- wheels -->
-			<left_joint>base_rear_left_wheel_joint</left_joint>
-			<right_joint>base_rear_right_wheel_joint</right_joint>
-			<!-- kinematics -->
-			<wheel_separation>0.6</wheel_separation>
-			<wheel_diameter>0.3</wheel_diameter>
-			<!-- limits
+  <gazebo reference="Ebox_link">
+    <material>Gazebo/Grey</material>
+  </gazebo>
+  <gazebo reference="rear_right_wheel_link">
+    <material>Gazebo/Blue</material>
+  </gazebo>
+  <gazebo reference="rear_left_wheel_link">
+    <material>Gazebo/Blue</material>
+  </gazebo>
+  <gazebo reference="front_right_wheel_link">
+    <material>Gazebo/Blue</material>
+    <mu1 value="0.1" />
+    <mu2 value="0.1" />
+  </gazebo>
+  <gazebo reference="front_left_wheel_link">
+    <material>Gazebo/Blue</material>
+    <mu1 value="0.1" />
+    <mu2 value="0.1" />
+  </gazebo>
+  <gazebo reference="lidar_link">
+    <material>Gazebo/Green</material>
+    <sensor name="lidar_sensor"
+      type="ray">
+      <pose>0 0 0 0 0 0</pose>
+      <visualize>true</visualize>
+      <update_rate>10.0</update_rate>
+      <ray>
+        <scan>
+          <horizontal>
+            <samples>720</samples>
+            <resolution>1</resolution>
+            <min_angle>-1.570796</min_angle>
+            <max_angle>1.570796</max_angle>
+          </horizontal>
+        </scan>
+        <range>
+          <min>0.15</min>
+          <max>10.0</max>
+          <resolution>0.01</resolution>
+        </range>
+        <noise>
+          <type>gaussian</type>
+          <!-- Noise parameters based on your specific sensor -->
+          <mean>0.0</mean>
+          <stddev>0.01</stddev>
+        </noise>
+      </ray>
+      <plugin name="lidar_sensor_plugin"
+        filename="libgazebo_ros_ray_sensor.so">
+        <ros>
+          <!-- Configure namespace and remap to publish to /lidar/pointcloud2 -->
+          <namespace>/lidar</namespace>
+          <remapping>~/out:=pointcloud2</remapping>
+        </ros>
+        <!-- Output as a PointCloud2, see above for other types -->
+        <output_type>sensor_msgs/PointCloud2</output_type>
+        <!-- Clip intensity values so all are above 100, optional -->
+        <min_intensity>100.0</min_intensity>
+        <!-- Frame id for header of output, defaults to sensor's parent link name -->
+        <frame_name>lidar_link</frame_name>
+      </plugin>
+    </sensor>
+  </gazebo>
+  <gazebo reference="imu_link">
+    <material>Gazebo/Green</material>
+    <sensor name="imu_sensor"
+      type="imu">
+      <plugin filename="libgazebo_ros_imu_sensor.so"
+        name="imu_plugin">
+        <ros>
+          <namespace>/imu_link</namespace>
+          <remapping>~/out:=imu</remapping>
+        </ros>
+        <initial_orientation_as_reference>false</initial_orientation_as_reference>
+      </plugin>
+      <always_on>true</always_on>
+      <update_rate>100</update_rate>
+      <visualize>true</visualize>
+      <imu>
+        <angular_velocity>
+          <x>
+            <noise type="gaussian">
+              <mean>0.0</mean>
+              <stddev>2e-4</stddev>
+              <bias_mean>0.0000075</bias_mean>
+              <bias_stddev>0.0000008</bias_stddev>
+            </noise>
+          </x>
+          <y>
+            <noise type="gaussian">
+              <mean>0.0</mean>
+              <stddev>2e-4</stddev>
+              <bias_mean>0.0000075</bias_mean>
+              <bias_stddev>0.0000008</bias_stddev>
+            </noise>
+          </y>
+          <z>
+            <noise type="gaussian">
+              <mean>0.0</mean>
+              <stddev>2e-4</stddev>
+              <bias_mean>0.0000075</bias_mean>
+              <bias_stddev>0.0000008</bias_stddev>
+            </noise>
+          </z>
+        </angular_velocity>
+        <linear_acceleration>
+          <x>
+            <noise type="gaussian">
+              <mean>0.0</mean>
+              <stddev>1.7e-2</stddev>
+              <bias_mean>0.1</bias_mean>
+              <bias_stddev>0.001</bias_stddev>
+            </noise>
+          </x>
+          <y>
+            <noise type="gaussian">
+              <mean>0.0</mean>
+              <stddev>1.7e-2</stddev>
+              <bias_mean>0.1</bias_mean>
+              <bias_stddev>0.001</bias_stddev>
+            </noise>
+          </y>
+          <z>
+            <noise type="gaussian">
+              <mean>0.0</mean>
+              <stddev>1.7e-2</stddev>
+              <bias_mean>0.1</bias_mean>
+              <bias_stddev>0.001</bias_stddev>
+            </noise>
+          </z>
+        </linear_acceleration>
+      </imu>
+    </sensor>
+  </gazebo>
+  <gazebo>
+    <plugin name="diff_drive_controller"
+      filename="libgazebo_ros_diff_drive.so">
+      <!-- Update rate in Hz -->
+      <update_rate>50</update_rate>
+      <!-- wheels -->
+      <left_joint>base_rear_left_wheel_joint</left_joint>
+      <right_joint>base_rear_right_wheel_joint</right_joint>
+      <!-- kinematics -->
+      <wheel_separation>0.6</wheel_separation>
+      <wheel_diameter>0.3</wheel_diameter>
+      <!-- limits
 			<max_wheel_torque>20</max_wheel_torque>
 			<max_wheel_acceleration>1.0</max_wheel_acceleration> -->
-			<!-- input
+      <!-- input
 			<command_topic>cmd_vel</command_topic> cms_vel is default-->
-			<!-- output -->
-            <!--keeping track of the robot based on wheel encoders-->
-			<publish_odom>true</publish_odom>
-			<publish_odom_tf>true</publish_odom_tf>
-			<publish_wheel_tf>true</publish_wheel_tf>
-			<odometry_topic>odom</odometry_topic>
-			<odometry_frame>odom</odometry_frame>
-			<robot_base_frame>base_link</robot_base_frame>
-		</plugin>
-	</gazebo>
+      <!-- output -->
+      <!--keeping track of the robot based on wheel encoders-->
+      <publish_odom>true</publish_odom>
+      <publish_odom_tf>true</publish_odom_tf>
+      <publish_wheel_tf>true</publish_wheel_tf>
+      <odometry_topic>odom</odometry_topic>
+      <odometry_frame>odom</odometry_frame>
+      <robot_base_frame>base_link</robot_base_frame>
+    </plugin>
+  </gazebo>
+  <gazebo reference="camera_link">
+    <material>Gazebo/Green</material>
+    <sensor name="depth_camera" type="depth">
+      <visualize>true</visualize>
+      <update_rate>30.0</update_rate>
+      <camera name="camera">
+        <horizontal_fov>1.50098</horizontal_fov>
+        <image>
+          <width>640</width>
+          <height>480</height>
+          <format>R8G8B8</format>
+        </image>
+        <clip>
+          <near>0.6</near>
+          <far>6</far>
+        </clip>
+      </camera>
+      <plugin name="depth_camera_controller" filename="libgazebo_ros_camera.so">
+        <baseline>0.2</baseline>
+        <alwaysOn>true</alwaysOn>
+        <updateRate>10.0</updateRate>
+        <frame_name>camera_depth_frame</frame_name>
+        <pointCloudCutoff>0.6</pointCloudCutoff>
+        <pointCloudCutoffMax>6.0</pointCloudCutoffMax>
+        <distortionK1>0</distortionK1>
+        <distortionK2>0</distortionK2>
+        <distortionK3>0</distortionK3>
+        <distortionT1>0</distortionT1>
+        <distortionT2>0</distortionT2>
+        <CxPrime>0</CxPrime>
+        <Cx>0</Cx>
+        <Cy>0</Cy>
+        <focalLength>0</focalLength>
+        <hackBaseline>0</hackBaseline>
+      </plugin>
+    </sensor>
+  </gazebo>
 </robot>

Commit message: added a motor controller for navigation and added a launch file for real test bot

File: src/test_bot_description/urdf/test_bot.xacro (robot description, xacro)
@@ -3,5 +3,5 @@
 	xmlns:xacro="http://www.ros.org/wiki/xacro">
 	<xacro:include filename="common_properties.xacro" />
-	<xacro:include filename="test_bot_gazebo.xacro" />
+	<!--<xacro:include filename="test_bot_gazebo.xacro" />-->
 	<xacro:property name="base_length"
 		value="0.8" />
@@ -25,5 +25,5 @@
 	<xacro:property name="lidar_height"
 		value="0.04" />
-	<xacro:property name="camera_length"
+	<!--<xacro:property name="camera_length"
 		value="0.015" />
 	<xacro:property name="camera_width"
@@ -36,5 +36,5 @@
 		value="0.02" />
 	<xacro:property name="camera_pole_height"
-		value="0.2" />
+		value="0.7" />-->
 	<link name="base_footprint" />
 	<link name="base_link">
@@ -115,5 +115,5 @@
 			rpy="0 0 0" />
 	</link>
-	<link name="camera_pole_link">
+	<!--<link name="camera_pole_link">
 		<visual>
 			<geometry>
@@ -137,5 +137,5 @@
 			xyz="0 0 0"
 			rpy="0 0 0" />
-	</link>
+	</link>-->
 	<link name="lidar_link">
 		<visual>
@@ -160,5 +160,5 @@
 			rpy="0 0 0" />
 	</link>
-	<link name="camera_link">
+	<!--<link name="camera_link">
 		<visual>
 			<origin xyz="0 0 0"
@@ -183,5 +183,5 @@
 			rpy="0 0 0" />
 	</link>
-	<link name="camera_depth_frame"/>
+	<link name="camera_depth_frame"/>-->
 	<link name="imu_link">
 		<visual>
@@ -249,5 +249,5 @@
 			rpy="0 0 0" />
 	</joint>
-	<joint name="base_camera_pole_joint"
+	<!--<joint name="base_camera_pole_joint"
 		type="fixed">
 		<parent link="base_link" />
@@ -255,5 +255,5 @@
 		<origin xyz="${(base_length / 2) - (2*lidar_radius) - (camera_pole_length/2)} 0 ${(base_height/2) + (camera_pole_height/2)}"
 			rpy="0 0 0" />
-	</joint>
+	</joint>-->
 	<joint name="base_lidar_joint"
 		type="fixed">
@@ -263,5 +263,5 @@
 			rpy="0 0 0" />
 	</joint>
-	<joint name="base_camera_joint"
+	<!--<joint name="base_camera_joint"
 		type="fixed">
 		<parent link="base_link" />
@@ -274,5 +274,5 @@
 		<parent link="camera_link"/>
 		<child link="camera_depth_frame"/>
-	  </joint>
+	</joint>-->
 	<joint name="base_imu_joint"
 		type="fixed">

File: src/test_bot_description/urdf/test_bot_gazebo.xacro (robot description, xacro)
@@ -54,5 +54,5 @@
           <remapping>~/out:=scan</remapping>
         </ros>
-        <!-- Output as a PointCloud2, see above for other types -->
+        <!-- Output as a laserscan, see above for other types -->
         <output_type>sensor_msgs/LaserScan</output_type>
         <!-- Clip intensity values so all are above 100, optional -->

Commit message: added hypothetical map and odom frame to urdf. added a test goal publisher to publish a random goal.

File: src/test_bot_description/urdf/test_bot.xacro (robot description, xacro)
@@ -38,4 +38,6 @@
 		value="0.7" />-->
 	<link name="base_footprint" />
+	<link name="odom" />
+	<link name="map" />
 	<link name="base_link">
 		<visual>
@@ -205,4 +207,18 @@
 			rpy="0 0 0" />
 	</link>
+	<joint name="odom_map"
+		type="fixed">
+		<parent link="map" />
+		<child link="odom" />
+		<origin xyz="0 0 0"
+			rpy="0 0 0" />
+	</joint>
+	<joint name="base_link_odom"
+		type="fixed">
+		<parent link="odom" />
+		<child link="base_link" />
+		<origin xyz="0 0 0"
+			rpy="0 0 0" />
+	</joint>
 	<joint name="base_joint"
 		type="fixed">

Commit message: test_goal_publisher works in gazebo at this point

File: src/test_bot_description/urdf/test_bot.xacro (robot description, xacro)
@@ -3,5 +3,5 @@
 	xmlns:xacro="http://www.ros.org/wiki/xacro">
 	<xacro:include filename="common_properties.xacro" />
-	<!--<xacro:include filename="test_bot_gazebo.xacro" />-->
+	<xacro:include filename="test_bot_gazebo.xacro" />
 	<xacro:property name="base_length"
 		value="0.8" />
@@ -25,5 +25,5 @@
 	<xacro:property name="lidar_height"
 		value="0.04" />
-	<!--<xacro:property name="camera_length"
+	<xacro:property name="camera_length"
 		value="0.015" />
 	<xacro:property name="camera_width"
@@ -36,8 +36,8 @@
 		value="0.02" />
 	<xacro:property name="camera_pole_height"
-		value="0.7" />-->
+		value="0.7" />
 	<link name="base_footprint" />
-	<link name="odom" />
-	<link name="map" />
+	<!--<link name="odom" />
+	<link name="map" />-->
 	<link name="base_link">
 		<visual>
@@ -117,5 +117,5 @@
 			rpy="0 0 0" />
 	</link>
-	<!--<link name="camera_pole_link">
+	<link name="camera_pole_link">
 		<visual>
 			<geometry>
@@ -139,5 +139,5 @@
 			xyz="0 0 0"
 			rpy="0 0 0" />
-	</link>-->
+	</link>
 	<link name="lidar_link">
 		<visual>
@@ -162,5 +162,5 @@
 			rpy="0 0 0" />
 	</link>
-	<!--<link name="camera_link">
+	<link name="camera_link">
 		<visual>
 			<origin xyz="0 0 0"
@@ -185,5 +185,5 @@
 			rpy="0 0 0" />
 	</link>
-	<link name="camera_depth_frame"/>-->
+	<link name="camera_depth_frame"/>
 	<link name="imu_link">
 		<visual>
@@ -207,5 +207,5 @@
 			rpy="0 0 0" />
 	</link>
-	<joint name="odom_map"
+	<!--<joint name="odom_map"
 		type="fixed">
 		<parent link="map" />
@@ -220,5 +220,5 @@
 		<origin xyz="0 0 0"
 			rpy="0 0 0" />
-	</joint>
+	</joint>-->
 	<joint name="base_joint"
 		type="fixed">
@@ -265,5 +265,5 @@
 			rpy="0 0 0" />
 	</joint>
-	<!--<joint name="base_camera_pole_joint"
+	<joint name="base_camera_pole_joint"
 		type="fixed">
 		<parent link="base_link" />
@@ -271,5 +271,5 @@
 		<origin xyz="${(base_length / 2) - (2*lidar_radius) - (camera_pole_length/2)} 0 ${(base_height/2) + (camera_pole_height/2)}"
 			rpy="0 0 0" />
-	</joint>-->
+	</joint>
 	<joint name="base_lidar_joint"
 		type="fixed">
@@ -279,5 +279,5 @@
 			rpy="0 0 0" />
 	</joint>
-	<!--<joint name="base_camera_joint"
+	<joint name="base_camera_joint"
 		type="fixed">
 		<parent link="base_link" />
@@ -290,5 +290,5 @@
 		<parent link="camera_link"/>
 		<child link="camera_depth_frame"/>
-	</joint>-->
+	</joint>
 	<joint name="base_imu_joint"
 		type="fixed">

Commit message: initial commit

File: src/test_bot_description/urdf/test_bot.xacro (robot description, xacro)
@@ -3,5 +3,5 @@
 	xmlns:xacro="http://www.ros.org/wiki/xacro">
 	<xacro:include filename="common_properties.xacro" />
-	<xacro:include filename="test_bot_gazebo.xacro" />
+	<!--<xacro:include filename="test_bot_gazebo.xacro" />-->
 	<xacro:property name="base_length"
 		value="0.8" />
@@ -25,5 +25,5 @@
 	<xacro:property name="lidar_height"
 		value="0.04" />
-	<xacro:property name="camera_length"
+	<!--<xacro:property name="camera_length"
 		value="0.015" />
 	<xacro:property name="camera_width"
@@ -36,5 +36,5 @@
 		value="0.02" />
 	<xacro:property name="camera_pole_height"
-		value="0.7" />
+		value="0.7" />-->
 	<link name="base_footprint" />
 	<!--<link name="odom" />
@@ -56,10 +56,10 @@
 				rpy="0 0 0" />
 		</collision>
-		<xacro:box_inertia m="7.0"
+		<!--<xacro:box_inertia m="7.0"
 			l="${base_length}"
 			w="${base_width}"
 			h="${base_height}"
 			xyz="0 0 ${base_height / 2}"
-			rpy="0 0 0" />
+			rpy="0 0 0" />-->
 	</link>
 	<xacro:macro name="wheel_link"
@@ -83,9 +83,9 @@
 					rpy="${pi / 2.0} 0 0" />
 			</collision>
-			<xacro:cylinder_inertia m="1.5"
+			<!--<xacro:cylinder_inertia m="1.5"
 				r="${wheel_radius}"
 				h="${wheel_length}"
 				xyz="0 0 0"
-				rpy="${pi / 2.0} 0 0" />
+				rpy="${pi / 2.0} 0 0" />-->
 		</link>
 	</xacro:macro>
@@ -110,12 +110,12 @@
 				rpy="0 0 0" />
 		</collision>
-		<xacro:box_inertia m="2.0"
+		<!--<xacro:box_inertia m="2.0"
 			l="${Ebox_length}"
 			w="${Ebox_width}"
 			h="${Ebox_height}"
 			xyz="0 0 0"
-			rpy="0 0 0" />
-	</link>
-	<link name="camera_pole_link">
+			rpy="0 0 0" />-->
+	</link>
+	<!--<link name="camera_pole_link">
 		<visual>
 			<geometry>
@@ -139,5 +139,5 @@
 			xyz="0 0 0"
 			rpy="0 0 0" />
-	</link>
+	</link>-->
 	<link name="lidar_link">
 		<visual>
@@ -156,11 +156,11 @@
 			</geometry>
 		</collision>
-		<xacro:cylinder_inertia m="0.1"
+		<!--<xacro:cylinder_inertia m="0.1"
 			r="${lidar_radius}"
 			h="${lidar_height}"
 			xyz="0 0 0"
-			rpy="0 0 0" />
-	</link>
-	<link name="camera_link">
+			rpy="0 0 0" />-->
+	</link>
+	<!--<link name="camera_link">
 		<visual>
 			<origin xyz="0 0 0"
@@ -207,5 +207,5 @@
 			rpy="0 0 0" />
 	</link>
-	<!--<joint name="odom_map"
+	<joint name="odom_map"
 		type="fixed">
 		<parent link="map" />
@@ -229,18 +229,18 @@
 	</joint>
 	<joint name="base_rear_right_wheel_joint"
-		type="continuous">
+		type="fixed">
 		<parent link="base_link" />
 		<child link="rear_right_wheel_link" />
 		<origin xyz="${-base_length / 4.0} ${-(base_width + wheel_length) / 2.0} 0"
 			rpy="0 0 0" />
-		<axis xyz="0 1 0" />
+		<!--<axis xyz="0 1 0" />-->
 	</joint>
 	<joint name="base_rear_left_wheel_joint"
-		type="continuous">
+		type="fixed">
 		<parent link="base_link" />
 		<child link="rear_left_wheel_link" />
 		<origin xyz="${-base_length / 4.0} ${(base_width + wheel_length) / 2.0} 0"
 			rpy="0 0 0" />
-		<axis xyz="0 1 0" />
+		<!--<axis xyz="0 1 0" />-->
 	</joint>
 	<joint name="base_front_right_wheel_joint"
@@ -265,5 +265,5 @@
 			rpy="0 0 0" />
 	</joint>
-	<joint name="base_camera_pole_joint"
+	<!--<joint name="base_camera_pole_joint"
 		type="fixed">
 		<parent link="base_link" />
@@ -271,5 +271,5 @@
 		<origin xyz="${(base_length / 2) - (2*lidar_radius) - (camera_pole_length/2)} 0 ${(base_height/2) + (camera_pole_height/2)}"
 			rpy="0 0 0" />
-	</joint>
+	</joint>-->
 	<joint name="base_lidar_joint"
 		type="fixed">
@@ -279,5 +279,5 @@
 			rpy="0 0 0" />
 	</joint>
-	<joint name="base_camera_joint"
+	<!--<joint name="base_camera_joint"
 		type="fixed">
 		<parent link="base_link" />
@@ -297,4 +297,4 @@
 		<origin xyz="0 0 ${base_height + 0.025}"
 			rpy="0 0 0" />
-	</joint>
+	</joint>-->
 </robot>
