Commit message: imu data is linked to odom and base_link

File: src/test_bot_description/urdf/test_bot.xacro (robot description, xacro)
@@ -25,5 +25,5 @@
 	<xacro:property name="lidar_height"
 		value="0.04" />
-	<!--<xacro:property name="camera_length"
+	<xacro:property name="camera_length"
 		value="0.015" />
 	<xacro:property name="camera_width"
@@ -31,5 +31,5 @@
 	<xacro:property name="camera_height"
 		value="0.022" />
-	<xacro:property name="camera_pole_length"
+	<!--<xacro:property name="camera_pole_length"
 		value="0.02" />
 	<xacro:property name="camera_pole_width"
@@ -185,5 +185,5 @@
 			rpy="0 0 0" />
 	</link>
-	<link name="camera_depth_frame"/>
+	<link name="camera_depth_frame"/>-->
 	<link name="imu_link">
 		<visual>
@@ -200,12 +200,12 @@
 			</geometry>
 		</collision>
-		<xacro:box_inertia m="0.1"
+		<!--<xacro:box_inertia m="0.1"
 			l="0.05"
 			w="0.05"
 			h="0.05"
 			xyz="0 0 0"
-			rpy="0 0 0" />
-	</link>
-	<joint name="odom_map"
+			rpy="0 0 0" />-->
+	</link>
+	<!--<joint name="odom_map"
 		type="fixed">
 		<parent link="map" />
@@ -290,5 +290,5 @@
 		<parent link="camera_link"/>
 		<child link="camera_depth_frame"/>
-	</joint>
+	</joint>-->
 	<joint name="base_imu_joint"
 		type="fixed">
@@ -297,4 +297,4 @@
 		<origin xyz="0 0 ${base_height + 0.025}"
 			rpy="0 0 0" />
-	</joint>-->
+	</joint>
 </robot>

Commit message: made base_footprint the parent of robot links. Odom is a child of base_footprint. Diff_Drive_Controller gazebo pluggin creates and publishes the odom tf. SLAM creates and publishes the map tf. SLAM works in gazebo at this point.

File: src/test_bot_description/urdf/test_bot.xacro (robot description, xacro)
@@ -3,5 +3,5 @@
 	xmlns:xacro="http://www.ros.org/wiki/xacro">
 	<xacro:include filename="common_properties.xacro" />
-	<!--<xacro:include filename="test_bot_gazebo.xacro" />-->
+	<xacro:include filename="test_bot_gazebo.xacro" />
 	<xacro:property name="base_length"
 		value="0.8" />
@@ -25,10 +25,10 @@
 	<xacro:property name="lidar_height"
 		value="0.04" />
-	<xacro:property name="camera_length"
+	<!--<xacro:property name="camera_length"
 		value="0.015" />
 	<xacro:property name="camera_width"
 		value="0.130" />
 	<xacro:property name="camera_height"
-		value="0.022" />
+		value="0.022" />-->
 	<!--<xacro:property name="camera_pole_length"
 		value="0.02" />
@@ -56,10 +56,10 @@
 				rpy="0 0 0" />
 		</collision>
-		<!--<xacro:box_inertia m="7.0"
+		<xacro:box_inertia m="7.0"
 			l="${base_length}"
 			w="${base_width}"
 			h="${base_height}"
 			xyz="0 0 ${base_height / 2}"
-			rpy="0 0 0" />-->
+			rpy="0 0 0" />
 	</link>
 	<xacro:macro name="wheel_link"
@@ -83,9 +83,9 @@
 					rpy="${pi / 2.0} 0 0" />
 			</collision>
-			<!--<xacro:cylinder_inertia m="1.5"
+			<xacro:cylinder_inertia m="1.5"
 				r="${wheel_radius}"
 				h="${wheel_length}"
 				xyz="0 0 0"
-				rpy="${pi / 2.0} 0 0" />-->
+				rpy="${pi / 2.0} 0 0" />
 		</link>
 	</xacro:macro>
@@ -110,10 +110,10 @@
 				rpy="0 0 0" />
 		</collision>
-		<!--<xacro:box_inertia m="2.0"
+		<xacro:box_inertia m="2.0"
 			l="${Ebox_length}"
 			w="${Ebox_width}"
 			h="${Ebox_height}"
 			xyz="0 0 0"
-			rpy="0 0 0" />-->
+			rpy="0 0 0" />
 	</link>
 	<!--<link name="camera_pole_link">
@@ -156,9 +156,9 @@
 			</geometry>
 		</collision>
-		<!--<xacro:cylinder_inertia m="0.1"
+		<xacro:cylinder_inertia m="0.1"
 			r="${lidar_radius}"
 			h="${lidar_height}"
 			xyz="0 0 0"
-			rpy="0 0 0" />-->
+			rpy="0 0 0" />
 	</link>
 	<!--<link name="camera_link">
@@ -200,10 +200,10 @@
 			</geometry>
 		</collision>
-		<!--<xacro:box_inertia m="0.1"
+		<xacro:box_inertia m="0.1"
 			l="0.05"
 			w="0.05"
 			h="0.05"
 			xyz="0 0 0"
-			rpy="0 0 0" />-->
+			rpy="0 0 0" />
 	</link>
 	<!--<joint name="odom_map"
@@ -223,24 +223,24 @@
 	<joint name="base_joint"
 		type="fixed">
-		<parent link="base_link" />
-		<child link="base_footprint" />
-		<origin xyz="0 0 ${-wheel_radius}"
+		<parent link="base_footprint" />
+		<child link="base_link" />
+		<origin xyz="0 0 ${wheel_radius}"
 			rpy="0 0 0" />
 	</joint>
 	<joint name="base_rear_right_wheel_joint"
-		type="fixed">
+		type="continuous">
 		<parent link="base_link" />
 		<child link="rear_right_wheel_link" />
 		<origin xyz="${-base_length / 4.0} ${-(base_width + wheel_length) / 2.0} 0"
 			rpy="0 0 0" />
-		<!--<axis xyz="0 1 0" />-->
+		<axis xyz="0 1 0" />
 	</joint>
 	<joint name="base_rear_left_wheel_joint"
-		type="fixed">
+		type="continuous">
 		<parent link="base_link" />
 		<child link="rear_left_wheel_link" />
 		<origin xyz="${-base_length / 4.0} ${(base_width + wheel_length) / 2.0} 0"
 			rpy="0 0 0" />
-		<!--<axis xyz="0 1 0" />-->
+		<axis xyz="0 1 0" />
 	</joint>
 	<joint name="base_front_right_wheel_joint"
@@ -277,5 +277,5 @@
 		<child link="lidar_link" />
 		<origin xyz="${(base_length/2) - lidar_radius} 0 ${base_height + (lidar_height/2)}"
-			rpy="0 0 -3.14" />
+			rpy="0 0 0" />
 	</joint>
 	<!--<joint name="base_camera_joint"

File: src/test_bot_description/urdf/test_bot_gazebo.xacro (robot description, xacro)
@@ -71,5 +71,5 @@
         <ros>
           <namespace>/imu_link</namespace>
-          <remapping>~/out:=imu</remapping>
+          <remapping>~/out:=camera/odom/sample</remapping>
         </ros>
         <initial_orientation_as_reference>false</initial_orientation_as_reference>
@@ -137,19 +137,12 @@
     <plugin name="diff_drive_controller"
       filename="libgazebo_ros_diff_drive.so">
-      <!-- Update rate in Hz -->
       <update_rate>50</update_rate>
-      <!-- wheels -->
       <left_joint>base_rear_left_wheel_joint</left_joint>
       <right_joint>base_rear_right_wheel_joint</right_joint>
-      <!-- kinematics -->
       <wheel_separation>0.6</wheel_separation>
       <wheel_diameter>0.3</wheel_diameter>
-      <!-- limits
 			<max_wheel_torque>20</max_wheel_torque>
-			<max_wheel_acceleration>1.0</max_wheel_acceleration> -->
-      <!-- input
-			<command_topic>cmd_vel</command_topic> cms_vel is default-->
-      <!-- output -->
-      <!--keeping track of the robot based on wheel encoders-->
+			<max_wheel_acceleration>1.0</max_wheel_acceleration>
+			<command_topic>cmd_vel</command_topic>
       <publish_odom>true</publish_odom>
       <publish_odom_tf>true</publish_odom_tf>
@@ -157,8 +150,8 @@
       <odometry_topic>odom</odometry_topic>
       <odometry_frame>odom</odometry_frame>
-      <robot_base_frame>base_link</robot_base_frame>
+      <robot_base_frame>base_footprint</robot_base_frame>
     </plugin>
   </gazebo>
-  <gazebo reference="camera_link">
+  <!--<gazebo reference="camera_link">
     <material>Gazebo/Green</material>
     <sensor name="depth_camera" type="depth">
@@ -196,4 +189,4 @@
       </plugin>
     </sensor>
-  </gazebo>
+  </gazebo>-->
 </robot>

Commit message: SLAM works on real test robot at this point. t265 camera creates and publishes odom to baselink tf and SLAM creates and publishes the map to odom tf.

File: src/test_bot_description/urdf/test_bot.xacro (robot description, xacro)
@@ -3,5 +3,5 @@
 	xmlns:xacro="http://www.ros.org/wiki/xacro">
 	<xacro:include filename="common_properties.xacro" />
-	<xacro:include filename="test_bot_gazebo.xacro" />
+	<!--<xacro:include filename="test_bot_gazebo.xacro" />-->
 	<xacro:property name="base_length"
 		value="0.8" />
@@ -186,5 +186,5 @@
 	</link>
 	<link name="camera_depth_frame"/>-->
-	<link name="imu_link">
+	<link name="camera_link">
 		<visual>
 			<geometry>
@@ -277,5 +277,5 @@
 		<child link="lidar_link" />
 		<origin xyz="${(base_length/2) - lidar_radius} 0 ${base_height + (lidar_height/2)}"
-			rpy="0 0 0" />
+			rpy="0 0 -3.14" />
 	</joint>
 	<!--<joint name="base_camera_joint"
@@ -291,8 +291,8 @@
 		<child link="camera_depth_frame"/>
 	</joint>-->
-	<joint name="base_imu_joint"
-		type="fixed">
-		<parent link="base_link" />
-		<child link="imu_link" />
+	<joint name="base_camera_joint"
+		type="fixed">
+		<parent link="base_link" />
+		<child link="camera_link" />
 		<origin xyz="0 0 ${base_height + 0.025}"
 			rpy="0 0 0" />

Commit message: tried using ros control, probably easier to write our own wheel odometry publisher

File: src/test_bot_description/urdf/test_bot.xacro (robot description, xacro)
@@ -3,13 +3,14 @@
 	xmlns:xacro="http://www.ros.org/wiki/xacro">
 	<xacro:include filename="common_properties.xacro" />
+	<!--<xacro:include filename="ros2_control.xacro" />-->
 	<!--<xacro:include filename="test_bot_gazebo.xacro" />-->
 	<xacro:property name="base_length"
-		value="0.8" />
+		value="0.915" />
 	<xacro:property name="base_width"
-		value="0.4" />
+		value="0.43" />
 	<xacro:property name="base_height"
 		value="0.08" />
 	<xacro:property name="wheel_radius"
-		value="0.12" />
+		value="0.1" />
 	<xacro:property name="wheel_length"
 		value="0.08" />
@@ -18,7 +19,7 @@
 		value="0.1" />
 	<xacro:property name="Ebox_width"
-		value="0.4" />
+		value="0.43" />
 	<xacro:property name="Ebox_height"
-		value="0.25" />
+		value="0.3" />
 	<xacro:property name="lidar_radius"
 		value="0.04" />
@@ -207,4 +208,7 @@
 			rpy="0 0 0" />
 	</link>
+	<link name="camera_fisheye1_optical_frame" />
+	<link name="camera_fisheye2_optical_frame" />
+	<link name="camera_pose_optical_frame" />
 	<!--<joint name="odom_map"
 		type="fixed">
@@ -298,3 +302,24 @@
 			rpy="0 0 0" />
 	</joint>
+	<joint name="base_camera_fisheye1_joint"
+		type="fixed">
+		<parent link="base_link" />
+		<child link="camera_fisheye1_optical_frame" />
+		<origin xyz="0 0 ${base_height + 0.025}"
+			rpy="0 0 0" />
+	</joint>
+	<joint name="base_camera_fisheye2_joint"
+		type="fixed">
+		<parent link="base_link" />
+		<child link="camera_fisheye2_optical_frame" />
+		<origin xyz="0 0 ${base_height + 0.025}"
+			rpy="0 0 0" />
+	</joint>
+	<joint name="base_camera_pose_frame"
+		type="fixed">
+		<parent link="base_link" />
+		<child link="camera_pose_optical_frame" />
+		<origin xyz="0 0 ${base_height + 0.025}"
+			rpy="0 0 0" />
+	</joint>
 </robot>

Commit message: Current code on the Jetson, I am currently working on a changes document due to the heavy amount of changes I made.

File: src/test_bot_description/urdf/test_bot.xacro (robot description, xacro)
@@ -14,5 +14,4 @@
 	<xacro:property name="wheel_length"
 		value="0.08" />
-	<!--Ebox = Electrical box-->
 	<xacro:property name="Ebox_length"
 		value="0.1" />
@@ -38,6 +37,4 @@
 		value="0.7" />-->
 	<link name="base_footprint" />
-	<!--<link name="odom" />
-	<link name="map" />-->
 	<link name="base_link">
 		<visual>
@@ -210,23 +207,9 @@
 	<link name="camera_fisheye2_optical_frame" />
 	<link name="camera_pose_optical_frame" />
-	<!--<joint name="odom_map"
-		type="fixed">
-		<parent link="map" />
-		<child link="odom" />
-		<origin xyz="0 0 0"
-			rpy="0 0 0" />
-	</joint>
-	<joint name="base_link_odom"
-		type="fixed">
-		<parent link="odom" />
-		<child link="base_link" />
-		<origin xyz="0 0 0"
-			rpy="0 0 0" />
-	</joint>-->
 	<joint name="base_joint"
 		type="fixed">
 		<parent link="base_footprint" />
 		<child link="base_link" />
-		<origin xyz="0 0 ${wheel_radius}"
+		<origin xyz="${base_length / 4.0} 0 ${wheel_radius}"
 			rpy="0 0 0" />
 	</joint>
@@ -265,5 +248,5 @@
 		<parent link="base_link" />
 		<child link="Ebox_link" />
-		<origin xyz="${(-base_length / 2) - (Ebox_length / 2)} 0 ${Ebox_height / 2}"
+		<origin xyz="${(-base_length / 2.0) - (Ebox_length / 2.0)} 0 ${Ebox_height / 2.0}"
 			rpy="0 0 0" />
 	</joint>
@@ -279,5 +262,5 @@
 		<parent link="base_link" />
 		<child link="lidar_link" />
-		<origin xyz="${(base_length/2) - lidar_radius} 0 ${base_height + (lidar_height/2)}"
+		<origin xyz="${(base_length/2.0) - lidar_radius} 0 ${base_height + (lidar_height/2.0)}"
 			rpy="0 0 -3.14" />
 	</joint>
@@ -298,5 +281,5 @@
 		<parent link="base_link" />
 		<child link="camera_link" />
-		<origin xyz="0 0 ${base_height + 0.025}"
+		<origin xyz="${-base_length / 4.0} 0 ${base_height + 0.025}"
 			rpy="0 0 0" />
 	</joint>
@@ -305,5 +288,5 @@
 		<parent link="base_link" />
 		<child link="camera_fisheye1_optical_frame" />
-		<origin xyz="0 0 ${base_height + 0.025}"
+		<origin xyz="${-base_length / 4.0} 0 ${base_height + 0.025}"
 			rpy="0 0 0" />
 	</joint>
@@ -312,5 +295,5 @@
 		<parent link="base_link" />
 		<child link="camera_fisheye2_optical_frame" />
-		<origin xyz="0 0 ${base_height + 0.025}"
+		<origin xyz="${-base_length / 4.0} 0 ${base_height + 0.025}"
 			rpy="0 0 0" />
 	</joint>
@@ -319,5 +302,5 @@
 		<parent link="base_link" />
 		<child link="camera_pose_optical_frame" />
-		<origin xyz="0 0 ${base_height + 0.025}"
+		<origin xyz="${-base_length / 4.0} 0 ${base_height + 0.025}"
 			rpy="0 0 0" />
 	</joint>

Commit message: Currently working on the real robot

File: src/test_bot_description/urdf/test_bot.xacro (robot description, xacro)
@@ -258,10 +258,10 @@
 			rpy="0 0 0" />
 	</joint>-->
+	<!--changed to 0, moved physical lidar to middle of robot-->
 	<joint name="base_lidar_joint"
 		type="fixed">
 		<parent link="base_link" />
 		<child link="lidar_link" />
-		<origin xyz="${(base_length/2.0) - lidar_radius} 0 ${base_height + (lidar_height/2.0)}"
-			rpy="0 0 -3.14" />
+		<origin xyz="0 0 ${base_height + (lidar_height/2.0)}" rpy="0 0 -3.14" />
 	</joint>
 	<!--<joint name="base_camera_joint"
