Commit message: Added a gazebo arena, configured urdf to work in gazebo, added a lidar that outputs a pointcloud, and added a launch pkg with a launch file that spawns our bot in gazebo

File: src/test_bot_description/urdf/common_properties.xacro (robot description, xacro)
@@ -7,3 +7,34 @@
         <color rgba="0.5 0.5 0.5 1" />
     </material>
+    <material name="green">
+        <color rgba="0.0 1 0.1 1" />
+    </material>
+    <xacro:macro name="box_inertia"
+        params="m l w h xyz rpy">
+        <inertial>
+            <origin xyz="${xyz}"
+                rpy="${rpy}" />
+            <mass value="${m}" />
+            <inertia ixx="${(m/12) * (h*h + l*l)}"
+                ixy="0"
+                ixz="0"
+                iyy="${(m/12) * (w*w + l*l)}"
+                iyz="0"
+                izz="${(m/12) * (w*w + h*h)}" />
+        </inertial>
+    </xacro:macro>
+    <xacro:macro name="cylinder_inertia"
+        params="m r h xyz rpy">
+        <inertial>
+            <origin xyz="${xyz}"
+                rpy="${rpy}" />
+            <mass value="${m}" />
+            <inertia ixx="${(m/12) * (3*r*r + h*h)}"
+                ixy="0"
+                ixz="0"
+                iyy="${(m/12) * (3*r*r + h*h)}"
+                iyz="0"
+                izz="${(m/2)*r*r}" />
+        </inertial>
+    </xacro:macro>
 </robot>

File: src/test_bot_description/urdf/test_bot.xacro (robot description, xacro)
@@ -1,80 +1,124 @@
 <?xml version="1.0"?>
-<robot name="test_bot" xmlns:xacro="http://www.ros.org/wiki/xacro">
-    <xacro:include filename="common_properties.xacro" />
-    <xacro:property name="base_length" value="1.0" />
-    <xacro:property name="base_width" value="0.5" />
-    <xacro:property name="base_height" value="0.08" />
-    <xacro:property name="wheel_radius" value="0.15" />
-    <xacro:property name="wheel_length" value="0.1" />
-    <xacro:property name="Ebox_length" value="0.1" /> <!--Ebox = Electrical box-->
-    <xacro:property name="Ebox_width" value="0.5" />
-    <xacro:property name="Ebox_height" value="0.3" />
-    <link name="base_footprint" />
-    <link name="base_link">
-        <visual>
-            <geometry>
-                <box size="${base_length} ${base_width} ${base_height}" />
-            </geometry>
-            <origin xyz="0 0 ${base_height / 2}" rpy="0 0 0" />
-            <material name="grey" />
-        </visual>
-    </link>
-    <xacro:macro name="wheel_link" params="prefix">
-        <link name="${prefix}_wheel_link">
-            <visual>
-                <geometry>
-                    <cylinder radius="${wheel_radius}" length="${wheel_length}" />
-                </geometry>
-                <origin xyz="0 0 0" rpy="${pi / 2.0} 0 0" />
-                <material name="blue" />
-            </visual>
-        </link>
-    </xacro:macro>
-    <xacro:wheel_link prefix="front_right" />
-    <xacro:wheel_link prefix="front_left" />
-    <xacro:wheel_link prefix="rear_right" />
-    <xacro:wheel_link prefix="rear_left" />
-    <link name="Ebox_link">
-        <visual>
-            <geometry>
-                <box size="${Ebox_length} ${Ebox_width} ${Ebox_height}" />
-            </geometry>
+<robot name="test_bot"
+	xmlns:xacro="http://www.ros.org/wiki/xacro">
+	<xacro:include filename="common_properties.xacro" />
+	<xacro:include filename="test_bot_gazebo.xacro" />
+	<xacro:property name="base_length" value="1.0" />
+	<xacro:property name="base_width" value="0.5" />
+	<xacro:property name="base_height" value="0.08" />
+	<xacro:property name="wheel_radius" value="0.15" />
+	<xacro:property name="wheel_length" value="0.1" />
+	<!--Ebox = Electrical box-->
+	<xacro:property name="Ebox_length" value="0.1" />
+	<xacro:property name="Ebox_width" value="0.5" />
+	<xacro:property name="Ebox_height" value="0.3" />
+    <xacro:property name="lidar_radius" value="0.04" />
+	<xacro:property name="lidar_height" value="0.04" />
+	<link name="base_footprint" />
+	<link name="base_link">
+		<visual>
+			<geometry>
+				<box size="${base_length} ${base_width} ${base_height}" />
+			</geometry>
+			<origin xyz="0 0 ${base_height / 2}" rpy="0 0 0" />
+			<material name="grey" />
+		</visual>
+		<collision>
+			<geometry>
+				<box size="${base_length} ${base_width} ${base_height}" />
+			</geometry>
+			<origin xyz="0 0 ${base_height / 2}" rpy="0 0 0" />
+		</collision>
+		<xacro:box_inertia m="7.0" l="${base_length}" w="${base_width}" h="${base_height}" xyz="0 0 ${base_height / 2}" rpy="0 0 0" />
+	</link>
+	<xacro:macro name="wheel_link" params="prefix">
+		<link name="${prefix}_wheel_link">
+			<visual>
+				<geometry>
+					<cylinder radius="${wheel_radius}" length="${wheel_length}" />
+				</geometry>
+				<origin xyz="0 0 0" rpy="${pi / 2.0} 0 0" />
+				<material name="blue" />
+			</visual>
+			<collision>
+				<geometry>
+					<cylinder radius="${wheel_radius}" length="${wheel_length}" />
+				</geometry>
+				<origin xyz="0 0 0" rpy="${pi / 2.0} 0 0" />
+			</collision>
+			<xacro:cylinder_inertia m="1.5" r="${wheel_radius}" h="${wheel_length}" xyz="0 0 0" rpy="${pi / 2.0} 0 0" />
+		</link>
+	</xacro:macro>
+	<xacro:wheel_link prefix="front_right" />
+	<xacro:wheel_link prefix="front_left" />
+	<xacro:wheel_link prefix="rear_right" />
+	<xacro:wheel_link prefix="rear_left" />
+	<link name="Ebox_link">
+		<visual>
+			<geometry>
+				<box size="${Ebox_length} ${Ebox_width} ${Ebox_height}" />
+			</geometry>
+			<origin xyz="0 0 0" rpy="0 0 0" />
+			<material name="grey" />
+		</visual>
+		<collision>
+			<geometry>
+				<box size="${Ebox_length} ${Ebox_width} ${Ebox_height}" />
+			</geometry>
+			<origin xyz="0 0 0" rpy="0 0 0" />
+		</collision>
+		<xacro:box_inertia m="2.0" l="${Ebox_length}" w="${Ebox_width}" h="${Ebox_height}" xyz="0 0 0" rpy="0 0 0" />
+	</link>
+	<link name="lidar_link">
+		<visual>
+			<geometry>
+				<cylinder radius="${lidar_radius}" length="${lidar_height}" />
+			</geometry>
             <origin xyz="0 0 0" rpy="0 0 0" />
-            <material name="grey" />
-        </visual>
-    </link>
-    <joint name="base_joint" type="fixed">
-        <parent link="base_footprint" />
-        <child link="base_link" />
-        <origin xyz="0 0 ${wheel_radius}" rpy="0 0 0"/>
-    </joint>
-    <joint name="base_rear_right_wheel_joint" type="continuous">
+			<material name="green" />
+		</visual>
+		<collision>
+			<geometry>
+				<cylinder radius="${lidar_radius}" length="${lidar_height}" />
+			</geometry>
+		</collision>
+		<xacro:cylinder_inertia m="0.1" r="${lidar_radius}" h="${lidar_height}" xyz="0 0 0" rpy="0 0 0" />
+	</link>
+	<joint name="base_joint" type="fixed">
+		<parent link="base_footprint" />
+		<child link="base_link" />
+		<origin xyz="0 0 ${wheel_radius}" rpy="0 0 0" />
+	</joint>
+	<joint name="base_rear_right_wheel_joint" type="continuous">
+		<parent link="base_link" />
+		<child link="rear_right_wheel_link" />
+		<origin xyz="${-base_length / 4.0} ${-(base_width + wheel_length) / 2.0} 0" rpy="0 0 0" />
+		<axis xyz="0 1 0" />
+	</joint>
+	<joint name="base_rear_left_wheel_joint" type="continuous">
+		<parent link="base_link" />
+		<child link="rear_left_wheel_link" />
+		<origin xyz="${-base_length / 4.0} ${(base_width + wheel_length) / 2.0} 0" rpy="0 0 0" />
+		<axis xyz="0 1 0" />
+	</joint>
+	<joint name="base_front_right_wheel_joint" type="fixed">
+		<parent link="base_link" />
+		<child link="front_right_wheel_link" />
+		<origin xyz="${base_length / 4.0} ${-(base_width + wheel_length) / 2.0} 0" rpy="0 0 0" />
+	</joint>
+	<joint name="base_front_left_wheel_joint" type="fixed">
+		<parent link="base_link" />
+		<child link="front_left_wheel_link" />
+		<origin xyz="${base_length / 4.0} ${(base_width + wheel_length) / 2.0} 0" rpy="0 0 0" />
+	</joint>
+	<joint name="base_Ebox_joint" type="fixed">
+		<parent link="base_link" />
+		<child link="Ebox_link" />
+		<origin xyz="${(-base_length / 2) - (Ebox_length / 2)} 0 ${Ebox_height / 2}" rpy="0 0 0" />
+	</joint>
+    <joint name="base_lidar_joint" type="fixed">
         <parent link="base_link" />
-        <child link="rear_right_wheel_link" />
-        <origin xyz="${-base_length / 4.0} ${-(base_width + wheel_length) / 2.0} 0" rpy="0 0 0" />
-        <axis xyz="0 1 0" />
-    </joint>
-    <joint name="base_rear_left_wheel_joint" type="continuous">
-        <parent link="base_link" />
-        <child link="rear_left_wheel_link" />
-        <origin xyz="${-base_length / 4.0} ${(base_width + wheel_length) / 2.0} 0" rpy="0 0 0" />
-        <axis xyz="0 1 0" />
-    </joint>
-    <joint name="base_front_right_wheel_joint" type="continuous">
-        <parent link="base_link" />
-        <child link="front_right_wheel_link" />
-        <origin xyz="${base_length / 4.0} ${-(base_width + wheel_length) / 2.0} 0" rpy="0 0 0" />
-        <axis xyz="0 1 0" />
-    </joint>
-    <joint name="base_front_left_wheel_joint" type="continuous">
-        <parent link="base_link" />
-        <child link="front_left_wheel_link" />
-        <origin xyz="${base_length / 4.0} ${(base_width + wheel_length) / 2.0} 0" rpy="0 0 0" />
-        <axis xyz="0 1 0" />
-    </joint>
-    <joint name="base_Ebox_joint" type="fixed">
-        <parent link="base_link" />
-        <child link="Ebox_link" />
-        <origin xyz="${-base_length / 2} 0 ${Ebox_height / 2}" rpy="0 0 0" />
+        <child link="lidar_link" />
+        <origin xyz="${(base_length/2) - lidar_radius} 0 ${base_height + (lidar_height/2)}" rpy="0 0 0" />
     </joint>
 </robot>

Commit message: This is the code that is to be ran on another computer, like a laptop. It shows everything in RViz.

File: src/test_bot_description/urdf/common_properties.xacro (robot description, xacro)
@@ -1,40 +1,15 @@
 <?xml version="1.0"?>
 <robot xmlns:xacro="http://www.ros.org/wiki/xacro">
-    <material name="blue">
-        <color rgba="0 0.1 1 1" />
+    <material name="light_grey">
+        <color rgba="0.61 0.61 0.61 1.0" />
     </material>
-    <material name="grey">
-        <color rgba="0.5 0.5 0.5 1" />
+    <material name="camera_grey">
+        <color rgba="0.81 0.81 0.81 1.0" />
     </material>
-    <material name="green">
-        <color rgba="0.0 1 0.1 1" />
+    <material name="black">
+        <color rgba="0.22 0.22 0.22 1.0" />
     </material>
-    <xacro:macro name="box_inertia"
-        params="m l w h xyz rpy">
-        <inertial>
-            <origin xyz="${xyz}"
-                rpy="${rpy}" />
-            <mass value="${m}" />
-            <inertia ixx="${(m/12) * (h*h + l*l)}"
-                ixy="0"
-                ixz="0"
-                iyy="${(m/12) * (w*w + l*l)}"
-                iyz="0"
-                izz="${(m/12) * (w*w + h*h)}" />
-        </inertial>
-    </xacro:macro>
-    <xacro:macro name="cylinder_inertia"
-        params="m r h xyz rpy">
-        <inertial>
-            <origin xyz="${xyz}"
-                rpy="${rpy}" />
-            <mass value="${m}" />
-            <inertia ixx="${(m/12) * (3*r*r + h*h)}"
-                ixy="0"
-                ixz="0"
-                iyy="${(m/12) * (3*r*r + h*h)}"
-                iyz="0"
-                izz="${(m/2)*r*r}" />
-        </inertial>
-    </xacro:macro>
+    <material name="white">
+        <color rgba="0.89 0.89 0.89 1.0" />
+    </material>
 </robot>

File: src/test_bot_description/urdf/test_bot.xacro (robot description, xacro)
@@ -3,60 +3,23 @@
 	xmlns:xacro="http://www.ros.org/wiki/xacro">
 	<xacro:include filename="common_properties.xacro" />
-	<!--<xacro:include filename="test_bot_gazebo.xacro" />-->
-	<xacro:property name="base_length"
-		value="0.915" />
-	<xacro:property name="base_width"
-		value="0.43" />
-	<xacro:property name="base_height"
-		value="0.08" />
-	<xacro:property name="wheel_radius"
-		value="0.1" />
-	<xacro:property name="wheel_length"
-		value="0.08" />
-	<xacro:property name="Ebox_length"
-		value="0.1" />
-	<xacro:property name="Ebox_width"
-		value="0.43" />
-	<xacro:property name="Ebox_height"
-		value="0.3" />
-	<xacro:property name="lidar_radius"
-		value="0.04" />
-	<xacro:property name="lidar_height"
-		value="0.04" />
-	<!--<xacro:property name="camera_length"
-		value="0.015" />
-	<xacro:property name="camera_width"
-		value="0.130" />
-	<xacro:property name="camera_height"
-		value="0.022" />-->
-	<!--<xacro:property name="camera_pole_length"
-		value="0.02" />
-	<xacro:property name="camera_pole_width"
-		value="0.02" />
-	<xacro:property name="camera_pole_height"
-		value="0.7" />-->
-	<link name="base_footprint" />
 	<link name="base_link">
 		<visual>
 			<geometry>
-				<box size="${base_length} ${base_width} ${base_height}" />
+				<mesh filename="package://test_bot_description/meshes/base_link.stl" />
 			</geometry>
-			<origin xyz="0 0 ${base_height / 2}"
+			<origin xyz="0 0 0"
 				rpy="0 0 0" />
-			<material name="grey" />
+			<material name="light_grey" />
 		</visual>
-		<collision>
+	</link>
+	<link name="ebox_link">
+		<visual>
 			<geometry>
-				<box size="${base_length} ${base_width} ${base_height}" />
+				<mesh filename="package://test_bot_description/meshes/ebox_link.stl" />
 			</geometry>
-			<origin xyz="0 0 ${base_height / 2}"
+			<origin xyz="0 0 0"
 				rpy="0 0 0" />
-		</collision>
-		<xacro:box_inertia m="7.0"
-			l="${base_length}"
-			w="${base_width}"
-			h="${base_height}"
-			xyz="0 0 ${base_height / 2}"
-			rpy="0 0 0" />
+			<material name="white" />
+		</visual>
 	</link>
 	<xacro:macro name="wheel_link"
@@ -65,24 +28,10 @@
 			<visual>
 				<geometry>
-					<cylinder radius="${wheel_radius}"
-						length="${wheel_length}" />
+					<mesh filename="package://test_bot_description/meshes/wheel_link.stl" />
 				</geometry>
 				<origin xyz="0 0 0"
 					rpy="${pi / 2.0} 0 0" />
-				<material name="blue" />
+				<material name="black" />
 			</visual>
-			<collision>
-				<geometry>
-					<cylinder radius="${wheel_radius}"
-						length="${wheel_length}" />
-				</geometry>
-				<origin xyz="0 0 0"
-					rpy="${pi / 2.0} 0 0" />
-			</collision>
-			<xacro:cylinder_inertia m="1.5"
-				r="${wheel_radius}"
-				h="${wheel_length}"
-				xyz="0 0 0"
-				rpy="${pi / 2.0} 0 0" />
 		</link>
 	</xacro:macro>
@@ -91,132 +40,29 @@
 	<xacro:wheel_link prefix="rear_right" />
 	<xacro:wheel_link prefix="rear_left" />
-	<link name="Ebox_link">
+	<link name="lidar_link">
 		<visual>
 			<geometry>
-				<box size="${Ebox_length} ${Ebox_width} ${Ebox_height}" />
+				<mesh filename="package://test_bot_description/meshes/lidar_link.stl" />
 			</geometry>
 			<origin xyz="0 0 0"
 				rpy="0 0 0" />
-			<material name="grey" />
+			<material name="black" />
 		</visual>
-		<collision>
+	</link>
+	<link name="camera_link">
+		<visual>
 			<geometry>
-				<box size="${Ebox_length} ${Ebox_width} ${Ebox_height}" />
+				<mesh filename="package://test_bot_description/meshes/camera_link.stl" />
 			</geometry>
 			<origin xyz="0 0 0"
 				rpy="0 0 0" />
-		</collision>
-		<xacro:box_inertia m="2.0"
-			l="${Ebox_length}"
-			w="${Ebox_width}"
-			h="${Ebox_height}"
-			xyz="0 0 0"
-			rpy="0 0 0" />
+			<material name="camera_grey" />
+		</visual>
 	</link>
-	<!--<link name="camera_pole_link">
-		<visual>
-			<geometry>
-				<box size="${camera_pole_length} ${camera_pole_width} ${camera_pole_height}" />
-			</geometry>
-			<origin xyz="0 0 0"
-				rpy="0 0 0" />
-			<material name="grey" />
-		</visual>
-		<collision>
-			<geometry>
-				<box size="${camera_pole_length} ${camera_pole_width} ${camera_pole_height}" />
-			</geometry>
-			<origin xyz="0 0 0"
-				rpy="0 0 0" />
-		</collision>
-		<xacro:box_inertia m="1.0"
-			l="${camera_pole_length}"
-			w="${camera_pole_width}"
-			h="${camera_pole_height}"
-			xyz="0 0 0"
-			rpy="0 0 0" />
-	</link>-->
-	<link name="lidar_link">
-		<visual>
-			<geometry>
-				<cylinder radius="${lidar_radius}"
-					length="${lidar_height}" />
-			</geometry>
-			<origin xyz="0 0 0"
-				rpy="0 0 0" />
-			<material name="green" />
-		</visual>
-		<collision>
-			<geometry>
-				<cylinder radius="${lidar_radius}"
-					length="${lidar_height}" />
-			</geometry>
-		</collision>
-		<xacro:cylinder_inertia m="0.1"
-			r="${lidar_radius}"
-			h="${lidar_height}"
-			xyz="0 0 0"
-			rpy="0 0 0" />
-	</link>
-	<!--<link name="camera_link">
-		<visual>
-			<origin xyz="0 0 0"
-				rpy="0 0 0" />
-			<geometry>
-				<box size="${camera_length} ${camera_width} ${camera_height}" />
-			</geometry>
-			<material name="green" />
-		</visual>
-		<collision>
-			<origin xyz="0 0 0"
-				rpy="0 0 0" />
-			<geometry>
-				<box size="${camera_length} ${camera_width} ${camera_height}" />
-			</geometry>
-		</collision>
-		<xacro:box_inertia m="0.1"
-			l="${camera_length}"
-			w="${camera_width}"
-			h="${camera_height}"
-			xyz="0 0 0"
-			rpy="0 0 0" />
-	</link>
-	<link name="camera_depth_frame"/>-->
-	<link name="camera_link">
-		<visual>
-			<geometry>
-				<box size="0.05 0.05 0.05" />
-			</geometry>
-			<origin xyz="0 0 0"
-				rpy="0 0 0" />
-			<material name="green" />
-		</visual>
-		<collision>
-			<geometry>
-				<box size="0.05 0.05 0.05" />
-			</geometry>
-		</collision>
-		<xacro:box_inertia m="0.1"
-			l="0.05"
-			w="0.05"
-			h="0.05"
-			xyz="0 0 0"
-			rpy="0 0 0" />
-	</link>
-	<link name="camera_fisheye1_optical_frame" />
-	<link name="camera_fisheye2_optical_frame" />
-	<link name="camera_pose_optical_frame" />
-	<joint name="base_joint"
-		type="fixed">
-		<parent link="base_footprint" />
-		<child link="base_link" />
-		<origin xyz="${base_length / 4.0} 0 ${wheel_radius}"
-			rpy="0 0 0" />
-	</joint>
 	<joint name="base_rear_right_wheel_joint"
 		type="continuous">
 		<parent link="base_link" />
 		<child link="rear_right_wheel_link" />
-		<origin xyz="${-base_length / 4.0} ${-(base_width + wheel_length) / 2.0} 0"
+		<origin xyz="-0.25 -0.1 0"
 			rpy="0 0 0" />
 		<axis xyz="0 1 0" />
@@ -226,13 +72,13 @@
 		<parent link="base_link" />
 		<child link="rear_left_wheel_link" />
-		<origin xyz="${-base_length / 4.0} ${(base_width + wheel_length) / 2.0} 0"
+		<origin xyz="-0.25 0.1 0"
 			rpy="0 0 0" />
 		<axis xyz="0 1 0" />
 	</joint>
 	<joint name="base_front_right_wheel_joint"
-		type="fixed">
+		type="continuous">
 		<parent link="base_link" />
 		<child link="front_right_wheel_link" />
-		<origin xyz="${base_length / 4.0} ${-(base_width + wheel_length) / 2.0} 0"
+		<origin xyz="0.25 -0.1 0"
 			rpy="0 0 0" />
 	</joint>
@@ -241,66 +87,24 @@
 		<parent link="base_link" />
 		<child link="front_left_wheel_link" />
-		<origin xyz="${base_length / 4.0} ${(base_width + wheel_length) / 2.0} 0"
+		<origin xyz="0.25 0.1 0"
 			rpy="0 0 0" />
 	</joint>
-	<joint name="base_Ebox_joint"
-		type="fixed">
-		<parent link="base_link" />
-		<child link="Ebox_link" />
-		<origin xyz="${(-base_length / 2.0) - (Ebox_length / 2.0)} 0 ${Ebox_height / 2.0}"
-			rpy="0 0 0" />
-	</joint>
-	<!--<joint name="base_camera_pole_joint"
-		type="fixed">
-		<parent link="base_link" />
-		<child link="camera_pole_link" />
-		<origin xyz="${(base_length / 2) - (2*lidar_radius) - (camera_pole_length/2)} 0 ${(base_height/2) + (camera_pole_height/2)}"
-			rpy="0 0 0" />
-	</joint>-->
-	<!--changed to 0, moved physical lidar to middle of robot-->
 	<joint name="base_lidar_joint"
 		type="fixed">
 		<parent link="base_link" />
 		<child link="lidar_link" />
-		<origin xyz="0 0 ${base_height + (lidar_height/2.0)}" rpy="0 0 -3.14" />
+		<origin xyz="0 0 0.18" rpy="0 0 3.14" />
 	</joint>
-	<!--<joint name="base_camera_joint"
+	<joint name="base_ebox_link"
 		type="fixed">
 		<parent link="base_link" />
-		<child link="camera_link" />
-		<origin xyz="${(base_length / 2) - (2*lidar_radius) - (camera_pole_length/2)} 0 ${(base_height/2) + (camera_pole_height) + (camera_height/2)}"
-			rpy="0 0 0" />
+		<child link="ebox_link" />
+		<origin xyz="0 0 0.125" rpy="0 0 0" />
 	</joint>
-	<joint name="camera_depth_joint" type="fixed">
-		<origin xyz="0 0 0" rpy="${-pi/2} 0 ${-pi/2}"/>
-		<parent link="camera_link"/>
-		<child link="camera_depth_frame"/>
-	</joint>-->
 	<joint name="base_camera_joint"
 		type="fixed">
 		<parent link="base_link" />
 		<child link="camera_link" />
-		<origin xyz="${-base_length / 4.0} 0 ${base_height + 0.025}"
-			rpy="0 0 0" />
-	</joint>
-	<joint name="base_camera_fisheye1_joint"
-		type="fixed">
-		<parent link="base_link" />
-		<child link="camera_fisheye1_optical_frame" />
-		<origin xyz="${-base_length / 4.0} 0 ${base_height + 0.025}"
-			rpy="0 0 0" />
-	</joint>
-	<joint name="base_camera_fisheye2_joint"
-		type="fixed">
-		<parent link="base_link" />
-		<child link="camera_fisheye2_optical_frame" />
-		<origin xyz="${-base_length / 4.0} 0 ${base_height + 0.025}"
-			rpy="0 0 0" />
-	</joint>
-	<joint name="base_camera_pose_frame"
-		type="fixed">
-		<parent link="base_link" />
-		<child link="camera_pose_optical_frame" />
-		<origin xyz="${-base_length / 4.0} 0 ${base_height + 0.025}"
+		<origin xyz="0.16 0 0.3"
 			rpy="0 0 0" />
 	</joint>
