Commit message: Added state estimation (particle filtering) and support for a second lidar. Still having issues with meshes loading in RViz, but it may just be my host computer.

File: lunabot/autonomous/test_bot_description/urdf/test_bot.xacro (robot description, xacro)
@@ -6,5 +6,5 @@
 		<visual>
 			<geometry>
-				<mesh filename="package://test_bot_description/meshes/base_link.stl" />
+				<mesh filename="file://$(find test_bot_description)/meshes/base_link.STL" />
 			</geometry>
 			<origin xyz="0 0 0"
@@ -16,5 +16,5 @@
 		<visual>
 			<geometry>
-				<mesh filename="package://test_bot_description/meshes/ebox_link.stl" />
+				<mesh filename="file://$(find test_bot_description)/meshes/ebox_link.STL" />
 			</geometry>
 			<origin xyz="0 0 0"
@@ -26,5 +26,5 @@
 		<visual>
 			<geometry>
-				<mesh filename="package://test_bot_description/meshes/wheel_link.stl" />
+				<mesh filename="file://$(find test_bot_description)/meshes/wheel_link.STL" />
 			</geometry>
 			<origin xyz="0 0 0"
@@ -36,5 +36,5 @@
 		<visual>
 			<geometry>
-				<mesh filename="package://test_bot_description/meshes/wheel_link.stl" />
+				<mesh filename="file://$(find test_bot_description)/meshes/wheel_link.STL" />
 			</geometry>
 			<origin xyz="0 0 0"
@@ -46,5 +46,5 @@
 		<visual>
 			<geometry>
-				<mesh filename="package://test_bot_description/meshes/wheel_link.stl" />
+				<mesh filename="file://$(find test_bot_description)/meshes/wheel_link.STL" />
 			</geometry>
 			<origin xyz="0 0 0"
@@ -56,5 +56,5 @@
 		<visual>
 			<geometry>
-				<mesh filename="package://test_bot_description/meshes/wheel_link.stl" />
+				<mesh filename="file://$(find test_bot_description)/meshes/wheel_link.STL" />
 			</geometry>
 			<origin xyz="0 0 0"
@@ -63,8 +63,18 @@
 		</visual>
 	</link>
-	<link name="lidar_link">
+	<link name="lidar1_link">
 		<visual>
 			<geometry>
-				<mesh filename="package://test_bot_description/meshes/lidar_link.stl" />
+				<mesh filename="file://$(find test_bot_description)/meshes/lidar_link.STL" />
+			</geometry>
+			<origin xyz="0 0 0"
+				rpy="0 0 0" />
+			<material name="black" />
+		</visual>
+	</link>
+	<link name="lidar2_link">
+		<visual>
+			<geometry>
+				<mesh filename="file://$(find test_bot_description)/meshes/lidar_link.STL" />
 			</geometry>
 			<origin xyz="0 0 0"
@@ -76,5 +86,5 @@
 		<visual>
 			<geometry>
-				<mesh filename="package://test_bot_description/meshes/camera_link.stl" />
+				<mesh filename="file://$(find test_bot_description)/meshes/camera_link.STL" />
 			</geometry>
 			<origin xyz="0 0 0"
@@ -113,9 +123,15 @@
 			rpy="0 0 0" />
 	</joint>
-	<joint name="base_lidar_joint"
+	<joint name="base_lidar1_joint"
 		type="fixed">
 		<parent link="base_link" />
-		<child link="lidar_link" />
+		<child link="lidar1_link" />
 		<origin xyz="0 0 0.19" rpy="0 0 3.14" />
+	</joint>
+	<joint name="base_lidar2_joint"
+		type="fixed">
+		<parent link="base_link" />
+		<child link="lidar2_link" />
+		<origin xyz="0.4572 0 0" rpy="0 0 3.14" />
 	</joint>
 	<joint name="base_ebox_link"
