Commit message: Particle filter works, also got both lidars working.

File: lunabot/autonomous/robot_description/urdf/test_bot.xacro (robot description, xacro)
@@ -133,5 +133,5 @@
 		<parent link="base_link" />
 		<child link="lidar2_link" />
-		<origin xyz="0.4572 0 0" rpy="0 0 3.14" />
+		<origin xyz="0.508 0 0" rpy="0 0 3.14" />
 	</joint>
 	<joint name="base_ebox_link"

Commit message: Fixed bug in particle_filter.cpp,  line 299 had theta first instead of x, so it was using incorrect values to update weights. Also added IMU data to particle_filter.cpp as well.

File: lunabot/autonomous/robot_description/urdf/test_bot.xacro (robot description, xacro)
@@ -6,5 +6,5 @@
 		<visual>
 			<geometry>
-				<mesh filename="file://$(find robot_description)/meshes/base_link.STL" />
+				<mesh filename="file:///$(find robot_description)/meshes/base_link.stl" />
 			</geometry>
 			<origin xyz="0 0 0"
@@ -16,5 +16,5 @@
 		<visual>
 			<geometry>
-				<mesh filename="file://$(find robot_description)/meshes/ebox_link.STL" />
+				<mesh filename="file:///$(find robot_description)/meshes/ebox_link.stl" />
 			</geometry>
 			<origin xyz="0 0 0"
@@ -26,5 +26,5 @@
 		<visual>
 			<geometry>
-				<mesh filename="file://$(find robot_description)/meshes/wheel_link.STL" />
+				<mesh filename="file:///$(find robot_description)/meshes/wheel_link.stl" />
 			</geometry>
 			<origin xyz="0 0 0"
@@ -36,5 +36,5 @@
 		<visual>
 			<geometry>
-				<mesh filename="file://$(find robot_description)/meshes/wheel_link.STL" />
+				<mesh filename="file:///$(find robot_description)/meshes/wheel_link.stl" />
 			</geometry>
 			<origin xyz="0 0 0"
@@ -46,5 +46,5 @@
 		<visual>
 			<geometry>
-				<mesh filename="file://$(find robot_description)/meshes/wheel_link.STL" />
+				<mesh filename="file:///$(find robot_description)/meshes/wheel_link.stl" />
 			</geometry>
 			<origin xyz="0 0 0"
@@ -56,5 +56,5 @@
 		<visual>
 			<geometry>
-				<mesh filename="file://$(find robot_description)/meshes/wheel_link.STL" />
+				<mesh filename="file:///$(find robot_description)/meshes/wheel_link.stl" />
 			</geometry>
 			<origin xyz="0 0 0"
@@ -66,5 +66,5 @@
 		<visual>
 			<geometry>
-				<mesh filename="file://$(find robot_description)/meshes/lidar_link.STL" />
+				<mesh filename="file:///$(find robot_description)/meshes/lidar_link.stl" />
 			</geometry>
 			<origin xyz="0 0 0"
@@ -76,5 +76,5 @@
 		<visual>
 			<geometry>
-				<mesh filename="file://$(find robot_description)/meshes/lidar_link.STL" />
+				<mesh filename="file:///$(find robot_description)/meshes/lidar_link.stl" />
 			</geometry>
 			<origin xyz="0 0 0"
@@ -86,5 +86,5 @@
 		<visual>
 			<geometry>
-				<mesh filename="file://$(find robot_description)/meshes/camera_link.STL" />
+				<mesh filename="file:///$(find robot_description)/meshes/camera_link.stl" />
 			</geometry>
 			<origin xyz="0 0 0"
@@ -133,5 +133,5 @@
 		<parent link="base_link" />
 		<child link="lidar2_link" />
-		<origin xyz="0.508 0 0" rpy="0 0 3.14" />
+		<origin xyz="0.48 0 0" rpy="0 0 3.14" />
 	</joint>
 	<joint name="base_ebox_link"

Commit message: Adjusted URDF and Navigation 2 parameters.

File: lunabot/autonomous/robot_description/urdf/test_bot.xacro (robot description, xacro)
@@ -97,5 +97,5 @@
 		<parent link="base_link" />
 		<child link="rear_right_wheel_link" />
-		<origin xyz="-0.25 -0.2 0"
+		<origin xyz="-0.19 -0.2 0"
 			rpy="0 0 0" />
 		<axis xyz="0 1 0" />
@@ -105,5 +105,5 @@
 		<parent link="base_link" />
 		<child link="rear_left_wheel_link" />
-		<origin xyz="-0.25 0.2 0"
+		<origin xyz="-0.19 0.2 0"
 			rpy="0 0 0" />
 		<axis xyz="0 1 0" />
@@ -113,5 +113,5 @@
 		<parent link="base_link" />
 		<child link="front_right_wheel_link" />
-		<origin xyz="0.25 -0.2 0"
+		<origin xyz="0.20 -0.2 0"
 			rpy="0 0 0" />
 	</joint>
@@ -120,5 +120,5 @@
 		<parent link="base_link" />
 		<child link="front_left_wheel_link" />
-		<origin xyz="0.25 0.2 0"
+		<origin xyz="0.20 0.2 0"
 			rpy="0 0 0" />
 	</joint>
@@ -133,5 +133,5 @@
 		<parent link="base_link" />
 		<child link="lidar2_link" />
-		<origin xyz="0.48 0 0" rpy="0 0 3.14" />
+		<origin xyz="0.38 0 0" rpy="0 0 3.14" />
 	</joint>
 	<joint name="base_ebox_link"

Commit message: Added T265 camera for extra odometry, added the S2L lidar, moved lidars to front and back of robot instead of having one in middle, adjusted Navigation 2 parameters, split intel_launch.py into multiple launch files to check sensor conditions before running RTAB-Map. Added install_dependencies.sh. Updated README.md.

File: lunabot/autonomous/robot_description/urdf/test_bot.xacro (robot description, xacro)
@@ -83,5 +83,15 @@
 		</visual>
 	</link>
-	<link name="camera_link">
+	<link name="d455_link">
+		<visual>
+			<geometry>
+				<mesh filename="file:///$(find robot_description)/meshes/camera_link.stl" />
+			</geometry>
+			<origin xyz="0 0 0"
+				rpy="0 0 0" />
+			<material name="camera_grey" />
+		</visual>
+	</link>
+	<link name="t265_link">
 		<visual>
 			<geometry>
@@ -127,5 +137,5 @@
 		<parent link="base_link" />
 		<child link="lidar1_link" />
-		<origin xyz="0 0 0.19" rpy="0 0 3.14" />
+		<origin xyz="0.374175 0 0" rpy="0 0 3.14" />
 	</joint>
 	<joint name="base_lidar2_joint"
@@ -133,5 +143,5 @@
 		<parent link="base_link" />
 		<child link="lidar2_link" />
-		<origin xyz="0.38 0 0" rpy="0 0 3.14" />
+		<origin xyz="-0.374175 0 0" rpy="0 0 0" />
 	</joint>
 	<joint name="base_ebox_link"
@@ -141,9 +151,16 @@
 		<origin xyz="0 0 0.125" rpy="0 0 0" />
 	</joint>
-	<joint name="base_camera_joint"
+	<joint name="base_d455_joint"
 		type="fixed">
 		<parent link="base_link" />
-		<child link="camera_link" />
-		<origin xyz="0.15 0 0.1"
+		<child link="d455_link" />
+		<origin xyz="0.169175 0 0.021"
+			rpy="0 0 0" />
+	</joint>
+	<joint name="base_t265_joint"
+		type="fixed">
+		<parent link="base_link" />
+		<child link="t265_link" />
+		<origin xyz="0.15 0 0.05"
 			rpy="0 0 0" />
 	</joint>
