Commit message: Changed scan input to scan_filtered, adjusted URDF.

File: description/urdf/test_bot.xacro (robot description, xacro)
@@ -127,5 +127,5 @@
 		<parent link="base_link" />
 		<child link="lidar1_link" />
-		<origin xyz="0.374175 0 0" rpy="0 0 3.14" />
+		<origin xyz="0.45 0 0" rpy="0 0 3.14" />
 	</joint>
 	<joint name="base_lidar2_joint"
@@ -145,5 +145,5 @@
 		<parent link="base_link" />
 		<child link="d455_link" />
-		<origin xyz="0.169175 0.18 0.21"
+		<origin xyz="0.20 0.10 0.21"
 			rpy="0 0 0" />
 	</joint>

Commit message: Updated meshes and re-aligned joints in URDF. Test bot was physically shortened.

File: description/urdf/test_bot.xacro (robot description, xacro)
@@ -66,8 +66,8 @@
 		<visual>
 			<geometry>
-				<mesh filename="file:///$(find description)/meshes/lidar_link.stl" />
+				<mesh filename="file:///$(find description)/meshes/lidar1_link.stl" />
 			</geometry>
 			<origin xyz="0 0 0"
-				rpy="0 0 0" />
+				rpy="0 0 ${pi / 2.0}" />
 			<material name="black" />
 		</visual>
@@ -76,5 +76,5 @@
 		<visual>
 			<geometry>
-				<mesh filename="file:///$(find description)/meshes/lidar_link.stl" />
+				<mesh filename="file:///$(find description)/meshes/lidar2_link.stl" />
 			</geometry>
 			<origin xyz="0 0 0"
@@ -88,7 +88,17 @@
 				<mesh filename="file:///$(find description)/meshes/camera_link.stl" />
 			</geometry>
-			<origin xyz="0 -0.18 0"
+			<origin xyz="0 -0.1 0"
 				rpy="0 0 0" />
 			<material name="camera_grey" />
+		</visual>
+	</link>
+	<link name="nuc_link">
+		<visual>
+			<geometry>
+				<mesh filename="file:///$(find description)/meshes/nuc_link.stl" />
+			</geometry>
+			<origin xyz="0 0 0"
+				rpy="${pi} 0 ${pi}" />
+			<material name="black" />
 		</visual>
 	</link>
@@ -113,5 +123,5 @@
 		<parent link="base_link" />
 		<child link="front_right_wheel_link" />
-		<origin xyz="0.20 -0.2 0"
+		<origin xyz="0.28 -0.2 0"
 			rpy="0 0 0" />
 	</joint>
@@ -120,5 +130,5 @@
 		<parent link="base_link" />
 		<child link="front_left_wheel_link" />
-		<origin xyz="0.20 0.2 0"
+		<origin xyz="0.28 0.2 0"
 			rpy="0 0 0" />
 	</joint>
@@ -127,5 +137,5 @@
 		<parent link="base_link" />
 		<child link="lidar1_link" />
-		<origin xyz="0.45 0 0" rpy="0 0 3.14" />
+		<origin xyz="0.3630625 0 0.02" rpy="0 0 ${pi}" />
 	</joint>
 	<joint name="base_lidar2_joint"
@@ -133,5 +143,5 @@
 		<parent link="base_link" />
 		<child link="lidar2_link" />
-		<origin xyz="-0.374175 0 0" rpy="0 0 0" />
+		<origin xyz="-0.3630625 0 0.04" rpy="0 0 0" />
 	</joint>
 	<joint name="base_ebox_link"
@@ -139,5 +149,5 @@
 		<parent link="base_link" />
 		<child link="ebox_link" />
-		<origin xyz="0 0 0.125" rpy="0 0 0" />
+		<origin xyz="0.04 0 0.125" rpy="0 0 0" />
 	</joint>
 	<joint name="base_d455_joint"
@@ -145,5 +155,12 @@
 		<parent link="base_link" />
 		<child link="d455_link" />
-		<origin xyz="0.20 0.10 0.21"
+		<origin xyz="0.1852625 0.10 0.12"
+			rpy="0 0 0" />
+	</joint>
+	<joint name="base_nuc_joint"
+		type="fixed">
+		<parent link="base_link" />
+		<child link="nuc_link" />
+		<origin xyz="-0.12 0.0 0.06"
 			rpy="0 0 0" />
 	</joint>

Commit message: Adjusted heights in URDF, robot is now above ground.

File: description/urdf/test_bot.xacro (robot description, xacro)
@@ -8,5 +8,5 @@
 				<mesh filename="file:///$(find description)/meshes/base_link.stl" />
 			</geometry>
-			<origin xyz="0 0 0"
+			<origin xyz="0 0 0.08"
 				rpy="0 0 0" />
 			<material name="light_grey" />
@@ -107,5 +107,5 @@
 		<parent link="base_link" />
 		<child link="rear_right_wheel_link" />
-		<origin xyz="-0.19 -0.2 0"
+		<origin xyz="-0.19 -0.2 0.08"
 			rpy="0 0 0" />
 		<axis xyz="0 1 0" />
@@ -115,5 +115,5 @@
 		<parent link="base_link" />
 		<child link="rear_left_wheel_link" />
-		<origin xyz="-0.19 0.2 0"
+		<origin xyz="-0.19 0.2 0.08"
 			rpy="0 0 0" />
 		<axis xyz="0 1 0" />
@@ -123,5 +123,5 @@
 		<parent link="base_link" />
 		<child link="front_right_wheel_link" />
-		<origin xyz="0.28 -0.2 0"
+		<origin xyz="0.28 -0.2 0.08"
 			rpy="0 0 0" />
 	</joint>
@@ -130,5 +130,5 @@
 		<parent link="base_link" />
 		<child link="front_left_wheel_link" />
-		<origin xyz="0.28 0.2 0"
+		<origin xyz="0.28 0.2 0.08"
 			rpy="0 0 0" />
 	</joint>
@@ -137,5 +137,5 @@
 		<parent link="base_link" />
 		<child link="lidar1_link" />
-		<origin xyz="0.3630625 0 0.02" rpy="0 0 ${pi}" />
+		<origin xyz="0.3630625 0 0.1" rpy="0 0 ${pi}" />
 	</joint>
 	<joint name="base_lidar2_joint"
@@ -143,5 +143,5 @@
 		<parent link="base_link" />
 		<child link="lidar2_link" />
-		<origin xyz="-0.3630625 0 0.04" rpy="0 0 0" />
+		<origin xyz="-0.3630625 0 0.12" rpy="0 0 0" />
 	</joint>
 	<joint name="base_ebox_link"
@@ -149,5 +149,5 @@
 		<parent link="base_link" />
 		<child link="ebox_link" />
-		<origin xyz="0.04 0 0.125" rpy="0 0 0" />
+		<origin xyz="0.04 0 0.205" rpy="0 0 0" />
 	</joint>
 	<joint name="base_d455_joint"
@@ -155,5 +155,5 @@
 		<parent link="base_link" />
 		<child link="d455_link" />
-		<origin xyz="0.1852625 0.10 0.12"
+		<origin xyz="0.1852625 0.10 0.20"
 			rpy="0 0 0" />
 	</joint>
@@ -162,5 +162,5 @@
 		<parent link="base_link" />
 		<child link="nuc_link" />
-		<origin xyz="-0.12 0.0 0.06"
+		<origin xyz="-0.12 0.0 0.14"
 			rpy="0 0 0" />
 	</joint>

Commit message: Updated URDF heights

File: description/urdf/test_bot.xacro (robot description, xacro)
@@ -8,5 +8,5 @@
 				<mesh filename="file:///$(find description)/meshes/base_link.stl" />
 			</geometry>
-			<origin xyz="0 0 0.08"
+			<origin xyz="0 0 0.085"
 				rpy="0 0 0" />
 			<material name="light_grey" />
@@ -107,5 +107,5 @@
 		<parent link="base_link" />
 		<child link="rear_right_wheel_link" />
-		<origin xyz="-0.19 -0.2 0.08"
+		<origin xyz="-0.19 -0.2 0.085"
 			rpy="0 0 0" />
 		<axis xyz="0 1 0" />
@@ -115,5 +115,5 @@
 		<parent link="base_link" />
 		<child link="rear_left_wheel_link" />
-		<origin xyz="-0.19 0.2 0.08"
+		<origin xyz="-0.19 0.2 0.085"
 			rpy="0 0 0" />
 		<axis xyz="0 1 0" />
@@ -123,5 +123,5 @@
 		<parent link="base_link" />
 		<child link="front_right_wheel_link" />
-		<origin xyz="0.28 -0.2 0.08"
+		<origin xyz="0.28 -0.2 0.085"
 			rpy="0 0 0" />
 	</joint>
@@ -130,5 +130,5 @@
 		<parent link="base_link" />
 		<child link="front_left_wheel_link" />
-		<origin xyz="0.28 0.2 0.08"
+		<origin xyz="0.28 0.2 0.085"
 			rpy="0 0 0" />
 	</joint>
@@ -137,5 +137,5 @@
 		<parent link="base_link" />
 		<child link="lidar1_link" />
-		<origin xyz="0.3630625 0 0.1" rpy="0 0 ${pi}" />
+		<origin xyz="0.3630625 0 0.105" rpy="0 0 ${pi}" />
 	</joint>
 	<joint name="base_lidar2_joint"
@@ -149,5 +149,5 @@
 		<parent link="base_link" />
 		<child link="ebox_link" />
-		<origin xyz="0.04 0 0.205" rpy="0 0 0" />
+		<origin xyz="0.04 0 0.21" rpy="0 0 0" />
 	</joint>
 	<joint name="base_d455_joint"
@@ -155,5 +155,5 @@
 		<parent link="base_link" />
 		<child link="d455_link" />
-		<origin xyz="0.1852625 0.10 0.20"
+		<origin xyz="0.1852625 0.10 0.205"
 			rpy="0 0 0" />
 	</joint>
@@ -162,5 +162,5 @@
 		<parent link="base_link" />
 		<child link="nuc_link" />
-		<origin xyz="-0.12 0.0 0.14"
+		<origin xyz="-0.12 0.0 0.145"
 			rpy="0 0 0" />
 	</joint>
