Commit message: Fixed transforms, adjusted ekf.yaml parameters, removed unnecessary static transformer in rs_multi_camera_launch.py, merged imu_rotator into one node instead of two.

File: lunabot/description/urdf/test_bot.xacro (robot description, xacro)
@@ -6,5 +6,5 @@
 		<visual>
 			<geometry>
-				<mesh filename="file:///$(find robot_description)/meshes/base_link.stl" />
+				<mesh filename="file:/$(find description)/meshes/base_link.stl" />
 			</geometry>
 			<origin xyz="0 0 0"
@@ -16,5 +16,5 @@
 		<visual>
 			<geometry>
-				<mesh filename="file:///$(find robot_description)/meshes/ebox_link.stl" />
+				<mesh filename="file:/$(find description)/meshes/ebox_link.stl" />
 			</geometry>
 			<origin xyz="0 0 0"
@@ -26,5 +26,5 @@
 		<visual>
 			<geometry>
-				<mesh filename="file:///$(find robot_description)/meshes/wheel_link.stl" />
+				<mesh filename="file://$(find description)/meshes/wheel_link.stl" />
 			</geometry>
 			<origin xyz="0 0 0"
@@ -36,5 +36,5 @@
 		<visual>
 			<geometry>
-				<mesh filename="file:///$(find robot_description)/meshes/wheel_link.stl" />
+				<mesh filename="file://$(find description)/meshes/wheel_link.stl" />
 			</geometry>
 			<origin xyz="0 0 0"
@@ -46,5 +46,5 @@
 		<visual>
 			<geometry>
-				<mesh filename="file:///$(find robot_description)/meshes/wheel_link.stl" />
+				<mesh filename="file://$(find description)/meshes/wheel_link.stl" />
 			</geometry>
 			<origin xyz="0 0 0"
@@ -56,5 +56,5 @@
 		<visual>
 			<geometry>
-				<mesh filename="file:///$(find robot_description)/meshes/wheel_link.stl" />
+				<mesh filename="file://$(find description)/meshes/wheel_link.stl" />
 			</geometry>
 			<origin xyz="0 0 0"
@@ -66,5 +66,5 @@
 		<visual>
 			<geometry>
-				<mesh filename="file:///$(find robot_description)/meshes/lidar_link.stl" />
+				<mesh filename="file://$(find description)/meshes/lidar_link.stl" />
 			</geometry>
 			<origin xyz="0 0 0"
@@ -76,5 +76,5 @@
 		<visual>
 			<geometry>
-				<mesh filename="file:///$(find robot_description)/meshes/lidar_link.stl" />
+				<mesh filename="file://$(find description)/meshes/lidar_link.stl" />
 			</geometry>
 			<origin xyz="0 0 0"
@@ -86,5 +86,5 @@
 		<visual>
 			<geometry>
-				<mesh filename="file:///$(find robot_description)/meshes/camera_link.stl" />
+				<mesh filename="file://$(find description)/meshes/camera_link.stl" />
 			</geometry>
 			<origin xyz="0 0 0"
@@ -96,5 +96,5 @@
 		<visual>
 			<geometry>
-				<mesh filename="file:///$(find robot_description)/meshes/camera_link.stl" />
+				<mesh filename="file://$(find description)/meshes/camera_link.stl" />
 			</geometry>
 			<origin xyz="0 0 0"

Commit message: Added updated robot meshes to description, edited robot_controller.cpp to have an "outdoor mode" designed for when the bigger, rough terrain wheels are on. Cleaned up hardware_monitor.cpp.

File: lunabot/description/urdf/test_bot.xacro (robot description, xacro)
@@ -8,5 +8,5 @@
 				<mesh filename="file:///$(find description)/meshes/base_link.stl" />
 			</geometry>
-			<origin xyz="0 0 0"
+			<origin xyz="0 0 0.085"
 				rpy="0 0 0" />
 			<material name="light_grey" />
@@ -66,8 +66,8 @@
 		<visual>
 			<geometry>
-				<mesh filename="file:///$(find description)/meshes/lidar_link.stl" />
+				<mesh filename="file:///$(find description)/meshes/lidar1_link.stl" />
 			</geometry>
 			<origin xyz="0 0 0"
-				rpy="0 0 0" />
+				rpy="0 0 ${pi / 2.0}" />
 			<material name="black" />
 		</visual>
@@ -76,5 +76,5 @@
 		<visual>
 			<geometry>
-				<mesh filename="file:///$(find description)/meshes/lidar_link.stl" />
+				<mesh filename="file:///$(find description)/meshes/lidar2_link.stl" />
 			</geometry>
 			<origin xyz="0 0 0"
@@ -88,7 +88,17 @@
 				<mesh filename="file:///$(find description)/meshes/camera_link.stl" />
 			</geometry>
-			<origin xyz="0 -0.18 0"
+			<origin xyz="0 -0.1 0"
 				rpy="0 0 0" />
 			<material name="camera_grey" />
+		</visual>
+	</link>
+	<link name="nuc_link">
+		<visual>
+			<geometry>
+				<mesh filename="file:///$(find description)/meshes/nuc_link.stl" />
+			</geometry>
+			<origin xyz="0 0 0"
+				rpy="${pi} 0 ${pi}" />
+			<material name="black" />
 		</visual>
 	</link>
@@ -97,5 +107,5 @@
 		<parent link="base_link" />
 		<child link="rear_right_wheel_link" />
-		<origin xyz="-0.19 -0.2 0"
+		<origin xyz="-0.19 -0.2 0.085"
 			rpy="0 0 0" />
 		<axis xyz="0 1 0" />
@@ -105,5 +115,5 @@
 		<parent link="base_link" />
 		<child link="rear_left_wheel_link" />
-		<origin xyz="-0.19 0.2 0"
+		<origin xyz="-0.19 0.2 0.085"
 			rpy="0 0 0" />
 		<axis xyz="0 1 0" />
@@ -113,5 +123,5 @@
 		<parent link="base_link" />
 		<child link="front_right_wheel_link" />
-		<origin xyz="0.20 -0.2 0"
+		<origin xyz="0.28 -0.2 0.085"
 			rpy="0 0 0" />
 	</joint>
@@ -120,5 +130,5 @@
 		<parent link="base_link" />
 		<child link="front_left_wheel_link" />
-		<origin xyz="0.20 0.2 0"
+		<origin xyz="0.28 0.2 0.085"
 			rpy="0 0 0" />
 	</joint>
@@ -127,5 +137,5 @@
 		<parent link="base_link" />
 		<child link="lidar1_link" />
-		<origin xyz="0.374175 0 0" rpy="0 0 3.14" />
+		<origin xyz="0.3630625 0 0.105" rpy="0 0 ${pi}" />
 	</joint>
 	<joint name="base_lidar2_joint"
@@ -133,5 +143,5 @@
 		<parent link="base_link" />
 		<child link="lidar2_link" />
-		<origin xyz="-0.374175 0 0" rpy="0 0 0" />
+		<origin xyz="-0.3630625 0 0.12" rpy="0 0 0" />
 	</joint>
 	<joint name="base_ebox_link"
@@ -139,5 +149,5 @@
 		<parent link="base_link" />
 		<child link="ebox_link" />
-		<origin xyz="0 0 0.125" rpy="0 0 0" />
+		<origin xyz="0.04 0 0.21" rpy="0 0 0" />
 	</joint>
 	<joint name="base_d455_joint"
@@ -145,5 +155,12 @@
 		<parent link="base_link" />
 		<child link="d455_link" />
-		<origin xyz="0.169175 0.18 0.21"
+		<origin xyz="0.1852625 0.1 0.2"
+			rpy="0 0 0" />
+	</joint>
+	<joint name="base_nuc_joint"
+		type="fixed">
+		<parent link="base_link" />
+		<child link="nuc_link" />
+		<origin xyz="-0.12 0.0 0.145"
 			rpy="0 0 0" />
 	</joint>
