Commit message: Renamed packages and removed lunabot folder, updated URDF with the bigger wheels.

File: lunabot_description/urdf/common_properties.xacro (robot description, xacro)
@@ -13,3 +13,6 @@
         <color rgba="0.89 0.89 0.89 1.0" />
     </material>
+     <material name="green">
+        <color rgba="0.03529412 0.32156863 0.24313725 1.0" />
+    </material>
 </robot>

File: lunabot_description/urdf/test_bot.xacro (robot description, xacro)
@@ -6,5 +6,5 @@
 		<visual>
 			<geometry>
-				<mesh filename="file:///$(find description)/meshes/base_link.stl" />
+				<mesh filename="file:///$(find lunabot_description)/meshes/base_link.stl" />
 			</geometry>
 			<origin xyz="0 0 0.085"
@@ -16,5 +16,5 @@
 		<visual>
 			<geometry>
-				<mesh filename="file:///$(find description)/meshes/ebox_link.stl" />
+				<mesh filename="file:///$(find lunabot_description)/meshes/ebox_link.stl" />
 			</geometry>
 			<origin xyz="0 0 0"
@@ -26,9 +26,9 @@
 		<visual>
 			<geometry>
-				<mesh filename="file:///$(find description)/meshes/wheel_link.stl" />
+				<mesh filename="file:///$(find lunabot_description)/meshes/wheel_link.stl" />
 			</geometry>
 			<origin xyz="0 0 0"
 				rpy="${pi / 2.0} 0 0" />
-			<material name="black" />
+			<material name="green" />
 		</visual>
 	</link>
@@ -36,9 +36,9 @@
 		<visual>
 			<geometry>
-				<mesh filename="file:///$(find description)/meshes/wheel_link.stl" />
+				<mesh filename="file:///$(find lunabot_description)/meshes/wheel_link.stl" />
 			</geometry>
 			<origin xyz="0 0 0"
-				rpy="${pi / 2.0} 0 0" />
-			<material name="black" />
+				rpy="${-pi / 2.0} 0 0" />
+			<material name="green" />
 		</visual>
 	</link>
@@ -46,9 +46,9 @@
 		<visual>
 			<geometry>
-				<mesh filename="file:///$(find description)/meshes/wheel_link.stl" />
+				<mesh filename="file:///$(find lunabot_description)/meshes/wheel_link.stl" />
 			</geometry>
 			<origin xyz="0 0 0"
 				rpy="${pi / 2.0} 0 0" />
-			<material name="black" />
+			<material name="green" />
 		</visual>
 	</link>
@@ -56,9 +56,9 @@
 		<visual>
 			<geometry>
-				<mesh filename="file:///$(find description)/meshes/wheel_link.stl" />
+				<mesh filename="file:///$(find lunabot_description)/meshes/wheel_link.stl" />
 			</geometry>
 			<origin xyz="0 0 0"
-				rpy="${pi / 2.0} 0 0" />
-			<material name="black" />
+				rpy="${-pi / 2.0} 0 0" />
+			<material name="green" />
 		</visual>
 	</link>
@@ -66,5 +66,5 @@
 		<visual>
 			<geometry>
-				<mesh filename="file:///$(find description)/meshes/lidar1_link.stl" />
+				<mesh filename="file:///$(find lunabot_description)/meshes/lidar1_link.stl" />
 			</geometry>
 			<origin xyz="0 0 0"
@@ -76,5 +76,5 @@
 		<visual>
 			<geometry>
-				<mesh filename="file:///$(find description)/meshes/lidar2_link.stl" />
+				<mesh filename="file:///$(find lunabot_description)/meshes/lidar2_link.stl" />
 			</geometry>
 			<origin xyz="0 0 0"
@@ -86,5 +86,5 @@
 		<visual>
 			<geometry>
-				<mesh filename="file:///$(find description)/meshes/camera_link.stl" />
+				<mesh filename="file:///$(find lunabot_description)/meshes/camera_link.stl" />
 			</geometry>
 			<origin xyz="0 -0.1 0"
@@ -96,5 +96,5 @@
 		<visual>
 			<geometry>
-				<mesh filename="file:///$(find description)/meshes/nuc_link.stl" />
+				<mesh filename="file:///$(find lunabot_description)/meshes/nuc_link.stl" />
 			</geometry>
 			<origin xyz="0 0 0"
@@ -107,5 +107,5 @@
 		<parent link="base_link" />
 		<child link="rear_right_wheel_link" />
-		<origin xyz="-0.19 -0.2 0.085"
+		<origin xyz="-0.19 -0.25 0.085"
 			rpy="0 0 0" />
 		<axis xyz="0 1 0" />
@@ -115,5 +115,5 @@
 		<parent link="base_link" />
 		<child link="rear_left_wheel_link" />
-		<origin xyz="-0.19 0.2 0.085"
+		<origin xyz="-0.19 0.25 0.085"
 			rpy="0 0 0" />
 		<axis xyz="0 1 0" />
@@ -123,5 +123,5 @@
 		<parent link="base_link" />
 		<child link="front_right_wheel_link" />
-		<origin xyz="0.28 -0.2 0.085"
+		<origin xyz="0.28 -0.25 0.085"
 			rpy="0 0 0" />
 	</joint>
@@ -130,5 +130,5 @@
 		<parent link="base_link" />
 		<child link="front_left_wheel_link" />
-		<origin xyz="0.28 0.2 0.085"
+		<origin xyz="0.28 0.25 0.085"
 			rpy="0 0 0" />
 	</joint>

Commit message: Renamed packages and updated README.md

File: lunabot_description/urdf/common_properties.xacro (robot description, xacro)
@@ -13,3 +13,6 @@
         <color rgba="0.89 0.89 0.89 1.0" />
     </material>
+    <material name="green">
+        <color rgba="0.03529412 0.32156863 0.24313725 1.0" />
+    </material>
 </robot>

File: lunabot_description/urdf/test_bot.xacro (robot description, xacro)
@@ -6,5 +6,5 @@
 		<visual>
 			<geometry>
-				<mesh filename="file:///$(find description)/meshes/base_link.stl" />
+				<mesh filename="file:///$(find lunabot_description)/meshes/base_link.stl" />
 			</geometry>
 			<origin xyz="0 0 0.085"
@@ -16,5 +16,5 @@
 		<visual>
 			<geometry>
-				<mesh filename="file:///$(find description)/meshes/ebox_link.stl" />
+				<mesh filename="file:///$(find lunabot_description)/meshes/ebox_link.stl" />
 			</geometry>
 			<origin xyz="0 0 0"
@@ -26,9 +26,9 @@
 		<visual>
 			<geometry>
-				<mesh filename="file:///$(find description)/meshes/wheel_link.stl" />
+				<mesh filename="file:///$(find lunabot_description)/meshes/wheel_link.stl" />
 			</geometry>
 			<origin xyz="0 0 0"
 				rpy="${pi / 2.0} 0 0" />
-			<material name="black" />
+			<material name="green" />
 		</visual>
 	</link>
@@ -36,9 +36,9 @@
 		<visual>
 			<geometry>
-				<mesh filename="file:///$(find description)/meshes/wheel_link.stl" />
+				<mesh filename="file:///$(find lunabot_description)/meshes/wheel_link.stl" />
 			</geometry>
 			<origin xyz="0 0 0"
-				rpy="${pi / 2.0} 0 0" />
-			<material name="black" />
+				rpy="${-pi / 2.0} 0 0" />
+			<material name="green" />
 		</visual>
 	</link>
@@ -46,9 +46,9 @@
 		<visual>
 			<geometry>
-				<mesh filename="file:///$(find description)/meshes/wheel_link.stl" />
+				<mesh filename="file:///$(find lunabot_description)/meshes/wheel_link.stl" />
 			</geometry>
 			<origin xyz="0 0 0"
 				rpy="${pi / 2.0} 0 0" />
-			<material name="black" />
+			<material name="green" />
 		</visual>
 	</link>
@@ -56,9 +56,9 @@
 		<visual>
 			<geometry>
-				<mesh filename="file:///$(find description)/meshes/wheel_link.stl" />
+				<mesh filename="file:///$(find lunabot_description)/meshes/wheel_link.stl" />
 			</geometry>
 			<origin xyz="0 0 0"
-				rpy="${pi / 2.0} 0 0" />
-			<material name="black" />
+				rpy="${-pi / 2.0} 0 0" />
+			<material name="green" />
 		</visual>
 	</link>
@@ -66,5 +66,5 @@
 		<visual>
 			<geometry>
-				<mesh filename="file:///$(find description)/meshes/lidar1_link.stl" />
+				<mesh filename="file:///$(find lunabot_description)/meshes/lidar1_link.stl" />
 			</geometry>
 			<origin xyz="0 0 0"
@@ -76,5 +76,5 @@
 		<visual>
 			<geometry>
-				<mesh filename="file:///$(find description)/meshes/lidar2_link.stl" />
+				<mesh filename="file:///$(find lunabot_description)/meshes/lidar2_link.stl" />
 			</geometry>
 			<origin xyz="0 0 0"
@@ -86,5 +86,5 @@
 		<visual>
 			<geometry>
-				<mesh filename="file:///$(find description)/meshes/camera_link.stl" />
+				<mesh filename="file:///$(find lunabot_description)/meshes/camera_link.stl" />
 			</geometry>
 			<origin xyz="0 -0.1 0"
@@ -96,5 +96,5 @@
 		<visual>
 			<geometry>
-				<mesh filename="file:///$(find description)/meshes/nuc_link.stl" />
+				<mesh filename="file:///$(find lunabot_description)/meshes/nuc_link.stl" />
 			</geometry>
 			<origin xyz="0 0 0"
@@ -107,5 +107,5 @@
 		<parent link="base_link" />
 		<child link="rear_right_wheel_link" />
-		<origin xyz="-0.19 -0.2 0.085"
+		<origin xyz="-0.19 -0.25 0.085"
 			rpy="0 0 0" />
 		<axis xyz="0 1 0" />
@@ -115,5 +115,5 @@
 		<parent link="base_link" />
 		<child link="rear_left_wheel_link" />
-		<origin xyz="-0.19 0.2 0.085"
+		<origin xyz="-0.19 0.25 0.085"
 			rpy="0 0 0" />
 		<axis xyz="0 1 0" />
@@ -123,5 +123,5 @@
 		<parent link="base_link" />
 		<child link="front_right_wheel_link" />
-		<origin xyz="0.28 -0.2 0.085"
+		<origin xyz="0.28 -0.25 0.085"
 			rpy="0 0 0" />
 	</joint>
@@ -130,5 +130,5 @@
 		<parent link="base_link" />
 		<child link="front_left_wheel_link" />
-		<origin xyz="0.28 0.2 0.085"
+		<origin xyz="0.28 0.25 0.085"
 			rpy="0 0 0" />
 	</joint>
@@ -155,5 +155,5 @@
 		<parent link="base_link" />
 		<child link="d455_link" />
-		<origin xyz="0.1852625 0.10 0.205"
+		<origin xyz="0.1852625 0.1 0.2"
 			rpy="0 0 0" />
 	</joint>
