Commit message: Updated URDF

File: lunabot_description/urdf/test_bot.xacro (robot description, xacro)
@@ -88,17 +88,7 @@
 				<mesh filename="file:///$(find lunabot_description)/meshes/camera_link.stl" />
 			</geometry>
-			<origin xyz="0 -0.1 0"
+			<origin xyz="0 -0.26 0"
 				rpy="0 0 0" />
 			<material name="camera_grey" />
-		</visual>
-	</link>
-	<link name="nuc_link">
-		<visual>
-			<geometry>
-				<mesh filename="file:///$(find lunabot_description)/meshes/nuc_link.stl" />
-			</geometry>
-			<origin xyz="0 0 0"
-				rpy="${pi} 0 ${pi}" />
-			<material name="black" />
 		</visual>
 	</link>
@@ -137,5 +127,5 @@
 		<parent link="base_link" />
 		<child link="lidar1_link" />
-		<origin xyz="0.3630625 0 0.105" rpy="0 0 ${pi}" />
+		<origin xyz="0.3630625 -0.1 0.105" rpy="0 0 ${pi}" />
 	</joint>
 	<joint name="base_lidar2_joint"
@@ -143,5 +133,5 @@
 		<parent link="base_link" />
 		<child link="lidar2_link" />
-		<origin xyz="-0.3630625 0 0.12" rpy="0 0 0" />
+		<origin xyz="0 0 0.26" rpy="0 0 ${pi}" />
 	</joint>
 	<joint name="base_ebox_link"
@@ -155,12 +145,5 @@
 		<parent link="base_link" />
 		<child link="d455_link" />
-		<origin xyz="0.1852625 0.1 0.2"
-			rpy="0 0 0" />
-	</joint>
-	<joint name="base_nuc_joint"
-		type="fixed">
-		<parent link="base_link" />
-		<child link="nuc_link" />
-		<origin xyz="-0.12 0.0 0.145"
+		<origin xyz="0.2 0.26 0.2"
 			rpy="0 0 0" />
 	</joint>

Commit message: Current code as of 2023-2024 competition.

File: lunabot_description/urdf/test_bot.xacro (robot description, xacro)
@@ -79,5 +79,5 @@
 			</geometry>
 			<origin xyz="0 0 0"
-				rpy="0 0 0" />
+				rpy="0 ${pi} 0" />
 			<material name="black" />
 		</visual>
@@ -88,5 +88,5 @@
 				<mesh filename="file:///$(find lunabot_description)/meshes/camera_link.stl" />
 			</geometry>
-			<origin xyz="0 -0.1 0"
+			<origin xyz="0 0.305 0"
 				rpy="0 0 0" />
 			<material name="camera_grey" />
@@ -137,5 +137,5 @@
 		<parent link="base_link" />
 		<child link="lidar1_link" />
-		<origin xyz="0.3630625 0 0.105" rpy="0 0 ${pi}" />
+		<origin xyz="0 0 0.71" rpy="0 0 ${pi}" />
 	</joint>
 	<joint name="base_lidar2_joint"
@@ -143,5 +143,5 @@
 		<parent link="base_link" />
 		<child link="lidar2_link" />
-		<origin xyz="-0.3630625 0 0.12" rpy="0 0 0" />
+		<origin xyz="0.305 0 0.12" rpy="0 ${pi} 0" />
 	</joint>
 	<joint name="base_ebox_link"
@@ -155,5 +155,5 @@
 		<parent link="base_link" />
 		<child link="d455_link" />
-		<origin xyz="0.1852625 0.1 0.2"
+		<origin xyz="0.305 0.1 0.2"
 			rpy="0 0 0" />
 	</joint>
